File: IDCSense/IDCSense.sch (KiCad schematic (older format))
At the start: 9 parts

Commit message: Update IDCSense
Parts:
- added C?: 1u, symbol C
- added C? (x7): 100n, symbol C
- added C? (x5): 10u, symbol C
- added D?: LED, symbol LED
- added D? (x3): D, symbol D
- added P?: nRF24L01+, symbol CONN_02X04
- added P?: I2C, symbol CONN_01X03
- added P?: Prog, symbol CONN_01X05
- added P?: IN, symbol CONN_01X03
- added P?: OUT, symbol CONN_01X03
- added R? (x2): 10, symbol R
- added R?: 100, symbol R
- added R? (x2): R, symbol R
- added R? (x2): 1k, symbol R
- added R?: nc, symbol R
- added R?: 0, symbol R
- added R?: 240, symbol R
- added R?: 390, symbol R
- added R?: 0.005, symbol R
- added R? (x2): 22k, symbol R
- added U?: PIC16F18323_QFN, symbol PIC16F18323_QFN
- added U?: MCP970x, symbol MCP970x
Connections:
- net labels added: +3.3V, /CS, CE, GND, GND_IN, GND_OUT, IRQ, MISO, MOSI, SCK, SCL, SDA, VIN, Vtemp
- wire segments 0 -> 121
Other:
- moved on the sheet: D?, P?, U?

Commit message: Update BancGeo
Parts:
- removed D?: D, symbol D
- removed P?: nRF24L01+, symbol CONN_02X04
- removed P? (x2): 6PCV-02-006, symbol CONN_01X02
- removed P?: I2C, symbol CONN_01X03
- removed P?: Prog, symbol CONN_01X05
- removed U?: PIC16F18323_QFN, symbol PIC16F18323_QFN
Changed lines of the file:
@@
 LIBS:YameLib
 LIBS:IDCSense-cache
-LIBS:IACSense-cache
 EELAYER 25 0
 EELAYER END
@@
 $EndDescr
 $Comp
-L PIC16F18323_QFN U?
-U 1 1 5676BE5E
-P 12000 -5200
-F 0 "U?" H 11600 -4650 60  0000 C CNN
-F 1 "PIC16F18323_QFN" H 12450 -6250 60  0000 C CNN
-F 2 "" H 12050 -5200 60  0000 C CNN
-F 3 "" H 12050 -5200 60  0000 C CNN
-	1    12000 -5200
-	1    0    0    -1
-$EndComp
-$Comp
 L LM317AT U?
 U 1 1 5676C508
@@
 	1    0    0    -1
 $EndComp
-$Comp
-L CONN_02X04 P?
-U 1 1 5676C6D0
-P 5400 -6000
-F 0 "P?" H 5400 -5750 50  0000 C CNN
-F 1 "nRF24L01+" H 5400 -6250 50  0000 C CNN
-F 2 "" H 5400 -7200 50  0000 C CNN
-F 3 "" H 5400 -7200 50  0000 C CNN
-	1    5400 -6000
-	-1   0    0    1
-$EndComp
-$Comp
-L CONN_01X02 P?
-U 1 1 5676C7FB
-P 4700 -4850
-F 0 "P?" H 4700 -4700 50  0000 C CNN
-F 1 "6PCV-02-006" V 4800 -4850 50  0000 C CNN
-F 2 "" H 4700 -4850 50  0000 C CNN
-F 3 "" H 4700 -4850 50  0000 C CNN
-	1    4700 -4850
-	1    0    0    -1
-$EndComp
-$Comp
-L CONN_01X02 P?
-U 1 1 5676C8B3
-P 4600 -6450
-F 0 "P?" H 4600 -6300 50  0000 C CNN
-F 1 "6PCV-02-006" V 4700 -6450 50  0000 C CNN
-F 2 "" H 4600 -6450 50  0000 C CNN
-F 3 "" H 4600 -6450 50  0000 C CNN
-	1    4600 -6450
-	1    0    0    -1
-$EndComp
-$Comp
-L CONN_01X03 P?
-U 1 1 5676C8C1
-P 6250 -6700
-F 0 "P?" H 6250 -6500 50  0000 C CNN
-F 1 "I2C" V 6350 -6700 50  0000 C CNN
-F 2 "" H 6250 -6700 50  0000 C CNN
-F 3 "" H 6250 -6700 50  0000 C CNN
-	1    6250 -6700
-	1    0    0    -1
-$EndComp
-$Comp
-L CONN_01X05 P?
-U 1 1 5676C91A
-P 6900 -6850
-F 0 "P?" H 6900 -6550 50  0000 C CNN
-F 1 "Prog" V 7000 -6850 50  0000 C CNN
-F 2 "" H 6900 -6850 50  0000 C CNN
-F 3 "" H 6900 -6850 50  0000 C CNN
-	1    6900 -6850
-	1    0    0    -1
-$EndComp
-$Comp
-L D D?
-U 1 1 5676CD3A
-P 7550 -4000
-F 0 "D?" H 7550 -3900 50  0000 C CNN
-F 1 "D" H 7550 -4100 50  0000 C CNN
-F 2 "" H 7550 -4000 50  0000 C CNN
-F 3 "" H 7550 -4000 50  0000 C CNN
-	1    7550 -4000
-	1    0    0    -1
-$EndComp
