File: BancGeo/BancGeo.kicad_pcb (KiCad board)
At the start: 2 copper layers, 127.5 x 96.5 mm, 121 parts, among them P1 Alim, P2 Batt, P3 CONN_01X05, P4 Capt1, P5 Capt2, P6 Capt3, P7 Capt4, P8 USB_D-, P9 USB_D+, Q1 2N7002E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

Commit message: Update BancGeo
Parts:
- added C36: 100n, Yame_library:SM0603-MR, F.Cu at (136.2, 147.6)
- moved C10 12.0 mm to (95.5, 133.3), turned to 270 degrees
- moved R7 11.8 mm to (93.0, 132.6), turned to 180 degrees
- moved R18 8.11 mm to (179.7, 141.0), turned to 90 degrees
- moved C20 6.12 mm to (106.5, 121.8)
- moved R22 6.12 mm to (105.7, 119.5)
- moved R23 6.12 mm to (105.0, 117.2)
- moved D2 5.67 mm to (171.3, 125.2)
- moved C19 3.29 mm to (177.7, 119.3)
- moved R21 3.21 mm to (177.7, 117.8)
- moved C17 3.06 mm to (172.6, 121.4)
- moved R20 3.00 mm to (174.9, 118.5)
- moved R19 2.88 mm to (172.5, 119.3)
- moved P8 1.96 mm to (83.6, 129.2)
- moved C15 1.85 mm to (172.6, 148.9)
- moved C12 1.85 mm to (172.6, 147.0)
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Connections:
- net Net-(C16-Pad1) renamed /Self_Out_2
- net Net-(C16-Pad2) renamed /TR_High_Side
- net Net-(Q3-Pad2) renamed /TR_Low_Side
- net Net-(R18-Pad1) renamed /Self_Out_1
- R9 pad 2: /+Vref1 -> /+Vref2
Routing:
- net Net-(P3-Pad1): track 0.00 -> 252.5 mm, vias 0 -> 3
- net /PWMin: track 0.00 -> 246.6 mm, vias 0 -> 4
- net Net-(R7-Pad2): track 0.00 -> 206.9 mm, vias 0 -> 2
- net /+Vref2: track 0.00 -> 144.2 mm, vias 0 -> 7
- net /SetPreChg: track 0.00 -> 112.4 mm, vias 0 -> 2
- net /SetTail: track 0.00 -> 108.8 mm, vias 0 -> 2
- net //Shdn: track 0.00 -> 95.0 mm, vias 0 -> 6
- net /SCL: track 0.00 -> 59.3 mm, vias 0 -> 6
- net /SDA: track 0.00 -> 58.5 mm, vias 0 -> 6
- net Net-(R22-Pad1): track 0.00 -> 52.1 mm
- net Net-(C19-Pad1): track 0.00 -> 43.4 mm, vias 0 -> 2
- net Net-(P3-Pad2): track 0.00 -> 37.7 mm, vias 0 -> 6
- net /VoffCHG: track 1.62 -> 38.0 mm, vias 0 -> 2
- net /Self_Out_1: track 0.00 -> 35.4 mm
- net /Vtemp: track 7.04 -> 41.1 mm, vias 1 -> 4
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- added copper zone on F.Cu, net /+12v
- added copper zone on F.Cu, net /+Vbat
- added copper zone on F.Cu, net /Self_Out_1
- added copper zone on F.Cu, net /Self_Out_2
- added copper zone on F.Cu, net /TR_High_Side
- added copper zone on F.Cu, net /TR_Low_Side

Commit message: Update BancGeo
Parts:
- added P10: GND, Yame_library:Test_Point_T_H, F.Cu at (78.0, 121.2)
- added Q6: 2N7002E, Yame_library:SOT23-MR, F.Cu at (166.3, 124.0)
- added R37: 100k, Yame_library:SM0603-MR, F.Cu at (163.3, 123.3)
- added R44: 100k, Yame_library:SM0603-MR, F.Cu at (122.0, 107.0)
- P1, P2: footprint Connect:PINHEAD1-2 -> Yame_library:PINHEAD1-2
- P4, P5, P6, P7: footprint Connect:PINHEAD1-3 -> Yame_library:PINHEAD1-3
- R1: value 10k -> 100k
- U3: value MCP6541 -> MCP6546
- moved Q1 51.3 mm to (167.2, 119.4)
- moved R1 50.5 mm to (163.2, 120.5)
- moved C13 23.3 mm to (168.6, 105.3), turned to 270 degrees
- moved U5 16.6 mm to (165.7, 108.6), turned to 180 degrees
- moved C7 16.2 mm to (168.6, 110.2)
- moved P8 3.38 mm to (81.5, 126.5)
- moved P9 1.89 mm to (78.0, 126.5)
Connections:
- Q1 pad 1: /VoffCHG -> Net-(Q1-Pad1)
- Q1 pad 3: Net-(Q1-Pad3) -> //Shdn
- R1 pad 2: /VoffCHG -> Net-(Q1-Pad1)
- R3 pad 2: Net-(Q1-Pad3) -> Net-(R3-Pad2)
- R4 pad 1: Net-(Q1-Pad3) -> Net-(R3-Pad2)
- REF** pad 1: (no net) -> GND (x6)
- U3 pad 3: Net-(Q1-Pad3) -> Net-(R3-Pad2)
- U6 pad 21: Net-(U6-Pad21) -> GND
- U7 pad 1: /VoffCHG -> //Shdn
- U7 pad 17: (no net) -> GND
- U9 pad 21: (no net) -> GND
Routing:
- net GND: track 0.00 -> 704.9 mm, vias 0 -> 86
- net /+5V: track 47.7 -> 438.1 mm, vias 2 -> 35
- net /+Vbat: track 56.7 -> 198.5 mm, vias 0 -> 14
- net //Shdn: track 95.0 -> 142.7 mm, vias 6 -> 10
- net /+3.3V: track 16.0 -> 59.6 mm
- net /VoffCHG: track 38.0 -> 0.00 mm, vias 2 -> 0
- net /+12v: track 14.9 -> 40.1 mm
- net /RDY: track 0.00 -> 23.3 mm, vias 0 -> 4
- net Net-(P8-Pad1): track 0.00 -> 10.4 mm
- net Net-(P3-Pad1): track 252.5 -> 242.3 mm
- net Net-(Q1-Pad3): track 7.95 -> 0.00 mm
- net Net-(P9-Pad1): track 0.00 -> 7.54 mm
- net Net-(Q3-Pad1): track 0.00 -> 7.30 mm, vias 0 -> 2
- net /Self_Out_1: track 35.4 -> 41.6 mm
- net Net-(Q1-Pad1): track 0.00 -> 4.79 mm
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- added copper zone on B.Cu, net GND
- added copper zone on F.Cu, net GND
Other:
- rule pad_to_mask_clearance: 0.2 -> 0.07
- board text added: "12V"
- board text added: "GP0"
- board text added: "GP1"
- board text added: "GP4"
- board text added: "GP5"
- board text added: "GP6"
- board text added: "GP7"
- board text added: "S0"
- board text added: "S1"
- board text added: "S2"
- board text added: "S3"
- board text added: "Vbat"
