File: BancGeo/BancGeo.sch (KiCad schematic (older format))
At the start: 126 parts, among them P1 Alim, P10 GND, P2 Batt, P3 CONN_01X05, P4 Capt1, P5 Capt2, P6 Capt3, P7 Capt4, P8 USB_D-, P9 USB_D+, Q1 2N7002E, Q2 PMV37EN2R, Q3 PMV37EN2R, Q4 2N7002E, Q5 2N7002E, Q6 2N7002E, SW1 SWITCH_BRIDE, SW2 SW_PUSH, T1 DRQ127-100-R, U1 MCP9700A, U10 MCP1754ST-3302E/CB, U12 LM4120IM5X-5.0/NOPB, U2 TC54VC4302ECB713, U3 MCP6546, U4 LM4120IM5X-5.0/NOPB, U5 MCP1754ST-5002E/CB, U6 MCP1631V-ML_QFN, U7 PIC16F18323_QFN, U8 ADS1115

Commit message: Update layout
Parts:
- removed Q?: P-MOS_SOIC, symbol P-MOS_SOIC
- removed R?: 100k, symbol R
- added K?: G5Q-1A, Relay_THT:Relay_SPST_Omron-G5Q-1A, symbol Relay:G5Q-1A
- C1, C10, C11, C12, C13, C14, C15, C16, C17, C18, C19, C2, C20, C21, C22, C23, C24, C25, C26, C27, C28, C29, C3, C30, C31, C32, C33, C34, C35, C36, C38, C4, C5, C6, C7, C8, C9: symbol C -> BancGeo-rescue:C
- D1, D10: renamed from D?; symbol DIODE_SCHOTTKY_3PIN -> BancGeo-rescue:DIODE_SCHOTTKY_3PIN
- D2: symbol D -> BancGeo-rescue:D
- D3, D4, D5, D6, D7, D8, D9: symbol LED-RESCUE-BancGeo -> BancGeo-rescue:LED-RESCUE-BancGeo
- P1, P2: symbol CONN_01X02 -> BancGeo-rescue:CONN_01X02
- P10, P8, P9: symbol CONN_01X01 -> BancGeo-rescue:CONN_01X01
- P3: symbol CONN_01X05 -> BancGeo-rescue:CONN_01X05
- P4, P5, P6, P7: symbol CONN_01X03 -> BancGeo-rescue:CONN_01X03
- Q1, Q2, Q3, Q4, Q5, Q6: symbol N-MOS_SOT23 -> BancGeo-rescue:N-MOS_SOT23
- R1, R10, R11, R12, R13, R14, R15, R16, R17, R18, R19, R2, R20, R21, R22, R23, R24, R25, R26, R27, R28, R29, R3, R30, R31, R32, R33, R34, R35, R36, R37, R38, R39, R4, R40, R41, R42, R43, R44, R5, R6, R7, R8, R9: symbol R -> BancGeo-rescue:R
- R46, R47: renamed from R?; symbol R -> BancGeo-rescue:R
- SW1: symbol SWITCH_BRIDE -> BancGeo-rescue:SWITCH_BRIDE
- SW2: symbol SW_PUSH -> BancGeo-rescue:SW_PUSH
- T1: symbol Coupled_Inductor -> BancGeo-rescue:Coupled_Inductor
- U1: symbol MCP970x -> BancGeo-rescue:MCP970x
- U10, U5: symbol MCP1754 -> BancGeo-rescue:MCP1754
- U11: renamed from U?; symbol HC-05_Bluetooth_Module -> BancGeo-rescue:HC-05_Bluetooth_Module
- U12, U4: symbol LM4120 -> BancGeo-rescue:LM4120
- U2: symbol TC54 -> BancGeo-rescue:TC54
- U3: symbol MCP6541 -> BancGeo-rescue:MCP6541
- U6: symbol MCP1631X-ML_QFN -> BancGeo-rescue:MCP1631X-ML_QFN
- U7: symbol PIC16F18323_QFN -> BancGeo-rescue:PIC16F18323_QFN
- U8: symbol ADS1115 -> BancGeo-rescue:ADS1115
- U9: renamed from U?; symbol MCP23008-QFN_PCKG -> BancGeo-rescue:MCP23008-QFN_PCKG
Connections:
- net labels added: GND1
- wire segments 434 -> 489
Other:
- moved on the sheet: P2, Q2

Commit message: Update lib : add VN7003ALH
Parts:
- C1, C10, C11, C12, C13, C14, C15, C16, C17, C18, C19, C2, C20, C21, C22, C23, C24, C25, C26, C27, C28, C29, C3, C30, C31, C32, C33, C34, C35, C36, C38, C4, C5, C6, C7, C8, C9: symbol BancGeo-rescue:C -> BancGeo-rescue:C-BancGeo-rescue
- D1, D10: symbol BancGeo-rescue:DIODE_SCHOTTKY_3PIN -> BancGeo-rescue:DIODE_SCHOTTKY_3PIN-BancGeo-rescue
- D2: symbol BancGeo-rescue:D -> BancGeo-rescue:D-BancGeo-rescue
- D3, D4, D5, D6, D7, D8, D9: symbol BancGeo-rescue:LED-RESCUE-BancGeo -> BancGeo-rescue:LED-RESCUE-BancGeo-BancGeo-rescue
- P1, P2: symbol BancGeo-rescue:CONN_01X02 -> BancGeo-rescue:CONN_01X02-BancGeo-rescue
- P10, P8, P9: symbol BancGeo-rescue:CONN_01X01 -> BancGeo-rescue:CONN_01X01-BancGeo-rescue
- P3: symbol BancGeo-rescue:CONN_01X05 -> BancGeo-rescue:CONN_01X05-BancGeo-rescue
- P4, P5, P6, P7: symbol BancGeo-rescue:CONN_01X03 -> BancGeo-rescue:CONN_01X03-BancGeo-rescue
- Q1, Q2, Q3, Q4, Q5, Q6: symbol BancGeo-rescue:N-MOS_SOT23 -> BancGeo-rescue:N-MOS_SOT23-BancGeo-rescue
- R1, R10, R11, R12, R13, R14, R15, R16, R17, R18, R19, R2, R20, R21, R22, R23, R24, R25, R26, R27, R28, R29, R3, R30, R31, R32, R33, R34, R35, R36, R37, R38, R39, R4, R40, R41, R42, R43, R44, R46, R47, R5, R6, R7, R8, R9: symbol BancGeo-rescue:R -> BancGeo-rescue:R-BancGeo-rescue
- SW1: symbol BancGeo-rescue:SWITCH_BRIDE -> BancGeo-rescue:SWITCH_BRIDE-BancGeo-rescue
- SW2: symbol BancGeo-rescue:SW_PUSH -> BancGeo-rescue:SW_PUSH-BancGeo-rescue
- T1: symbol BancGeo-rescue:Coupled_Inductor -> BancGeo-rescue:Coupled_Inductor-BancGeo-rescue
- U1: symbol BancGeo-rescue:MCP970x -> BancGeo-rescue:MCP970x-BancGeo-rescue
- U10, U5: symbol BancGeo-rescue:MCP1754 -> BancGeo-rescue:MCP1754-BancGeo-rescue
- U11: symbol BancGeo-rescue:HC-05_Bluetooth_Module -> BancGeo-rescue:HC-05_Bluetooth_Module-BancGeo-rescue
- U12, U4: symbol BancGeo-rescue:LM4120 -> BancGeo-rescue:LM4120-BancGeo-rescue
- U2: symbol BancGeo-rescue:TC54 -> BancGeo-rescue:TC54-BancGeo-rescue
- U3: symbol BancGeo-rescue:MCP6541 -> BancGeo-rescue:MCP6541-BancGeo-rescue
- U6: symbol BancGeo-rescue:MCP1631X-ML_QFN -> BancGeo-rescue:MCP1631X-ML_QFN-BancGeo-rescue
- U7: symbol BancGeo-rescue:PIC16F18323_QFN -> BancGeo-rescue:PIC16F18323_QFN-BancGeo-rescue
- U8: symbol BancGeo-rescue:ADS1115 -> BancGeo-rescue:ADS1115-BancGeo-rescue
- U9: symbol BancGeo-rescue:MCP23008-QFN_PCKG -> BancGeo-rescue:MCP23008-QFN_PCKG-BancGeo-rescue

Commit message: Add X-pressure design
Connections:
- wire segments 489 -> 490
