File: IACSense/IACSense.sch (KiCad schematic (older format))
At the start: 9 parts

Commit message: modif IACSense project
Parts:
- added C?: C, symbol C
- added C?: CP, symbol CP
- added D?: ZENER, symbol ZENER
- added D?: MB8S, symbol Diode_Bridge
- added F?: FUSE, symbol FUSE
- added R? (x2): R, symbol R
- added VR?: VR, symbol VR
Connections:
- new net: C?.2, R?.1, R?.2, VR?.2
- new net: C?.1, D?.4, R?.1
- new net: C?.1, D?.1 (K), D?.3 (+)
- new net: C?.2, D?.1 (-), D?.2 (A)
- new net: D?.2, F?.2, VR?.1
- new net L: F?.1
- new net N: R?.2
Other:
- note added: "iso1541"
- moved on the sheet: D?, P?
Changed lines of the file:
@@
 LIBS:contrib
 LIBS:valves
-LIBS:IDBox
+LIBS:YameLib
 LIBS:IACSense-cache
 EELAYER 25 0
@@
 L CONN_02X04 P?
 U 1 1 5676C6D0
-P 2050 2050
-F 0 "P?" H 2050 2300 50  0000 C CNN
-F 1 "nRF24L01+" H 2050 1800 50  0000 C CNN
-F 2 "" H 2050 850 50  0000 C CNN
-F 3 "" H 2050 850 50  0000 C CNN
-	1    2050 2050
+P 2300 2200
+F 0 "P?" H 2300 2450 50  0000 C CNN
+F 1 "nRF24L01+" H 2300 1950 50  0000 C CNN
+F 2 "" H 2300 1000 50  0000 C CNN
+F 3 "" H 2300 1000 50  0000 C CNN
+	1    2300 2200
 	-1   0    0    1
 $EndComp
@@
 L D D?
 U 1 1 5676CD3A
-P 4200 4050
-F 0 "D?" H 4200 4150 50  0000 C CNN
-F 1 "D" H 4200 3950 50  0000 C CNN
-F 2 "" H 4200 4050 50  0000 C CNN
-F 3 "" H 4200 4050 50  0000 C CNN
-	1    4200 4050
+P 3750 2950
+F 0 "D?" H 3750 3050 50  0000 C CNN
+F 1 "D" H 3750 2850 50  0000 C CNN
+F 2 "" H 3750 2950 50  0000 C CNN
+F 3 "" H 3750 2950 50  0000 C CNN
+	1    3750 2950
 	1    0    0    -1
 $EndComp
@@
 	1    0    0    -1
 $EndComp
+$Comp
+L R R?
+U 1 1 56C0DBF2
+P 1400 6350
+F 0 "R?" V 1480 6350 50  0000 C CNN
+F 1 "R" V 1400 6350 50  0000 C CNN
+F 2 "" V 1330 6350 30  0000 C CNN
+F 3 "" H 1400 6350 30  0000 C CNN
+	1    1400 6350
+	0    1    1    0
+$EndComp
+$Comp
+L C C?
+U 1 1 56C0DC53
+P 2050 6350
+F 0 "C?" H 2075 6450 50  0000 L CNN
+F 1 "C" H 2075 6250 50  0000 L CNN
+F 2 "" H 2088 6200 30  0000 C CNN
+F 3 "" H 2050 6350 60  0000 C CNN
+	1    2050 6350
+	0    1    1    0
+$EndComp
+$Comp
+L ZENER D?
+U 1 1 56C0DCAC
+P 4550 6200
+F 0 "D?" H 4550 6300 50  0000 C CNN
+F 1 "ZENER" H 4550 6100 50  0000 C CNN
+F 2 "" H 4550 6200 60  0000 C CNN
+F 3 "" H 4550 6200 60  0000 C CNN
+	1    4550 6200
+	0    1    1    0
+$EndComp
+$Comp
+L CP C?
+U 1 1 56C0DD81
+P 5300 6200
+F 0 "C?" H 5325 6300 50  0000 L CNN
+F 1 "CP" H 5325 6100 50  0000 L CNN
+F 2 "" H 5338 6050 30  0000 C CNN
+F 3 "" H 5300 6200 60  0000 C CNN
+	1    5300 6200
+	1    0    0    -1
+$EndComp
+$Comp
+L VR VR?
+U 1 1 56C0DDD0
+P 1700 5950
+F 0 "VR?" V 1760 5904 50  0000 C TNN
+F 1 "VR" V 1700 5950 50  0000 C CNN
+F 2 "" H 1700 5950 60  0000 C CNN
+F 3 "" H 1700 5950 60  0000 C CNN
+	1    1700 5950
+	1    0    0    -1
+$EndComp
+$Comp
+L R R?
+U 1 1 56C0DE33
+P 2050 6800
+F 0 "R?" V 2130 6800 50  0000 C CNN
+F 1 "R" V 2050 6800 50  0000 C CNN
+F 2 "" V 1980 6800 30  0000 C CNN
+F 3 "" H 2050 6800 30  0000 C CNN
+	1    2050 6800
+	0    1    1    0
+$EndComp
+$Comp
+L FUSE F?
+U 1 1 56C0DE8E
+P 1350 5450
+F 0 "F?" H 1450 5500 50  0000 C CNN
+F 1 "FUSE" H 1250 5400 50  0000 C CNN
+F 2 "" H 1350 5450 60  0000 C CNN
+F 3 "" H 1350 5450 60  0000 C CNN
+	1    1350 5450
+	1    0    0    -1
+$EndComp
+$Comp
+L Diode_Bridge D?
+U 1 1 56C0DEF7
+P 3400 6350
+F 0 "D?" H 3400 6400 50  0000 C CNN
+F 1 "MB8S" H 3400 6300 50  0000 C CNN
+F 2 "" H 3400 6350 60  0000 C CNN
+F 3 "" H 3400 6350 60  0000 C CNN
+	1    3400 6350
+	0    -1   -1   0
+$EndComp
+Wire Wire Line
+	1250 6350 850  6350
+Wire Wire Line
+	1100 5450 750  5450
+Text Label 750  5450 0    60   ~ 0
+L
+Text Label 850  6350 0    60   ~ 0
+N
+Wire Wire Line
+	3400 7050 5300 7050
+Wire Wire Line
+	5300 7050 5300 6350
+Wire Wire Line
+	4550 6400 4550 7050
+Connection ~ 4550 7050
+Wire Wire Line
+	3400 5650 5300 5650
+Wire Wire Line
+	5300 5650 5300 6050
+Wire Wire Line
+	4550 6000 4550 5650
+Connection ~ 4550 5650
+Wire Wire Line
+	1600 5450 4100 5450
+Wire Wire Line
+	4100 5450 4100 6350
+Wire Wire Line
+	1550 6350 1900 6350
+Wire Wire Line
+	1700 6200 1700 6350
+Connection ~ 1700 6350
+Wire Wire Line
+	2200 6350 2700 6350
+Wire Wire Line
+	1900 6800 1850 6800
+Wire Wire Line
+	1850 6800 1850 6350
+Connection ~ 1850 6350
+Wire Wire Line
+	2250 6350 2250 6800
+Wire Wire Line
+	2250 6800 2200 6800
+Connection ~ 2250 6350
+Wire Wire Line
+	1700 5700 1700 5450
+Connection ~ 1700 5450
+Text Notes 5650 1300 0    60   ~ 0
+iso1541
 $EndSCHEMATC

Commit message: Update IACSense
Parts:
- removed D?: D, symbol D
- removed P? (x2): 6PCV-02-006, symbol CONN_01X02
- removed U?: LM317AT, TO-220, symbol LM317AT
- added C? (x4): 33n, symbol C
- added C? (x2): C, symbol C
- added C? (x7): 100n, symbol C
- added C? (x5): 10u, symbol C
- added D?: LED, symbol LED
- added FB? (x4): LI0805H151R-10, symbol FILTER
- added P? (x2): CONN_01X03, symbol CONN_01X03
- added P?: zcd, symbol CONN_01X01
- added P?: event, symbol CONN_01X01
- added R?: 0.002, symbol R
- added R?: 2.49, symbol R
- added R? (x8): 1k, symbol R
- added R? (x2): 499k, symbol R
- added R? (x2): R, symbol R
- added R?: 100, symbol R
- added R?: 33, symbol R
- added U?: MCP1754, symbol MCP1754
- added U?: MCP970x, symbol MCP970x
- added Y?: 4MHz, symbol Crystal_Small
- C?: value C -> 0.68uF_X2_B32922C3684M
- D?: value ZENER -> 4.7V
- D?: symbol Diode_Bridge -> Diode_Bridge-RESCUE-IACSense
- F?: value FUSE -> FC-230
- R?: value R -> 100_0.5W_1206
- VR?: value VR -> ERZ-E05A361
Connections:
- net labels added: 3.3A, 3.3D, GND, Ground, Line, Neutral, SCL, SDA, Vtemp
- net labels removed: L, N
- wire segments 18 -> 188
Other:
- note added: "18*11*18.5"
- note added: "BZX85C4V7\nZMM5230B\n"
- note removed: "iso1541"
- moved on the sheet: C?, D?, F?, P?, R?, U?, VR?

Commit message: Update layout
Parts:
- added R?: nc, symbol R
- added R?: 0, symbol R
Connections:
- net labels added: /CS, CE, IRQ, MISO, MOSI, SCK
- wire segments 188 -> 176
Other:
- moved on the sheet: P?

Commit message: update IACSense
Parts:
- C1, C12, C13, C14, C16, C17, C2, C20, C4, C5, C6, C7, C8: renamed from C?; footprint (none) -> Yame_library:SM0603-MR
- C10: renamed from C?; footprint (none) -> Capacitors_ThroughHole:C_Radial_D14_L25_P5
- C11, C15, C18, C19, C9: renamed from C?; footprint (none) -> Yame_library:SM0805-MR
- D2: renamed from D?; value 4.7V -> BZX85C4V7; footprint (none) -> Diodes_ThroughHole:Diode_DO-41_SOD81_Horizontal_RM10
- D3: renamed from D?; footprint (none) -> LEDs:LED_0603
- F1: renamed from F?; footprint (none) -> Fuse_Holders_and_Fuses:Fuseholder5x20_horiz_open_inline_Type-I
- FB1, FB2, FB3, FB4: renamed from FB?; footprint (none) -> Yame_library:SM0805-MR
- P3, P4: renamed from P?; footprint (none) -> Yame_library:Test_Point_T_H
- P5: renamed from P?; footprint (none) -> Yame_library:HE10_14-5C-2.54-MR
- R1, R10, R11, R12, R13, R14, R15, R16, R17, R18, R19, R2, R20, R3, R4, R5, R6, R7, R8, R9: renamed from R?; footprint (none) -> Yame_library:SM0603-MR
- U1: renamed from U?; footprint (none) -> Housings_DFN_QFN:QFN-28-1EP_5x5mm_Pitch0.5mm
- U2: renamed from U?; footprint (none) -> Yame_library:SOT23-MR
- U3: renamed from U?; footprint (none) -> TO_SOT_Packages_THT:TO-220_Neutral123_Vertical
- U4: renamed from U?; footprint (none) -> Housings_DFN_QFN:QFN-16-1EP_4x4mm_Pitch0.65mm
- Y1: renamed from Y?; footprint (none) -> Crystals:Q_49U3HMS
- gave numbers to parts that had none: 7

Commit message: update IACSense
Parts:
- D1: footprint (none) -> Yame_library:MBxS
- P6: footprint (none) -> Yame_library:HE10_14-2x4C-2.54-MR
- P7: footprint (none) -> Yame_library:HE10_14-3C-2.54-MR
Changed lines of the file:
@@
 F 0 "P6" H 10100 4650 50  0000 C CNN
 F 1 "nRF24L01+" H 10100 4150 50  0000 C CNN
-F 2 "" H 10100 3200 50  0001 C CNN
+F 2 "Yame_library:HE10_14-2x4C-2.54-MR" H 10100 3200 50  0001 C CNN
 F 3 "" H 10100 3200 50  0000 C CNN
 	1    10100 4400
@@
 F 0 "P7" H 10650 1150 50  0000 C CNN
 F 1 "I2C" V 10750 950 50  0000 C CNN
-F 2 "" H 10650 950 50  0001 C CNN
+F 2 "Yame_library:HE10_14-3C-2.54-MR" H 10650 950 50  0001 C CNN
 F 3 "" H 10650 950 50  0000 C CNN
 	1    10650 950
@@
 F 0 "D1" H 4300 6400 50  0000 C CNN
 F 1 "MB8S" H 4300 6300 50  0000 C CNN
-F 2 "" H 4300 6350 60  0001 C CNN
+F 2 "Yame_library:MBxS" H 4300 6350 60  0001 C CNN
 F 3 "" H 4300 6350 60  0000 C CNN
 	1    4300 6350

Commit message: Update IACSense
Parts:
- removed F1: FC-230, Fuse_Holders_and_Fuses:Fuseholder5x20_horiz_open_inline_Type-I, symbol FUSE
- added F1: 0751.0062, Yame_library:Fuse_5x20, symbol FUSE_CLIP_5x20
- C3: footprint (none) -> Yame_library:X2_15mm
- D2: footprint Diodes_ThroughHole:Diode_DO-41_SOD81_Horizontal_RM10 -> Yame_library:DO-204AL
- FB1, FB2, FB3, FB4: value LI0805H151R-10 -> BLM18AG102SN1D; footprint Yame_library:SM0805-MR -> Yame_library:SM0603-MR
- P1, P2: footprint (none) -> Yame_library:Conn3_Term
- R1: value 0.002 -> LRMAM1206-R002FT5; footprint Yame_library:SM0603-MR -> Yame_library:SM1206-MR
- VR1: footprint (none) -> Yame_library:VR_5mm
Connections:
- wire segments 176 -> 180
Changed lines of the file:
@@
 F 0 "C3" H 2975 6450 50  0000 L CNN
 F 1 "0.68uF_X2_B32922C3684M" V 2800 6100 50  0000 L CNN
-F 2 "" H 2988 6200 30  0001 C CNN
+F 2 "Yame_library:X2_15mm" H 2988 6200 30  0001 C CNN
 F 3 "" H 2950 6350 60  0000 C CNN
 	1    2950 6350
@@
 F 0 "D2" H 5450 6300 50  0000 C CNN
 F 1 "BZX85C4V7" H 5450 6100 50  0000 C CNN
-F 2 "Diodes_ThroughHole:Diode_DO-41_SOD81_Horizontal_RM10" H 5450 6200 60  0001 C CNN
+F 2 "Yame_library:DO-204AL" H 5450 6200 60  0001 C CNN
 F 3 "" H 5450 6200 60  0000 C CNN
 	1    5450 6200
@@
 F 0 "VR1" V 860 5604 50  0000 C TNN
 F 1 "ERZ-E05A361" V 700 5650 50  0000 C CNN
-F 2 "" H 800 5650 60  0001 C CNN
+F 2 "Yame_library:VR_5mm" H 800 5650 60  0001 C CNN
 F 3 "" H 800 5650 60  0000 C CNN
 	1    800  5650
@@
 $EndComp
 $Comp
-L FUSE F1
-U 1 1 56C0DE8E
-P 1550 5450
-F 0 "F1" H 1650 5500 50  0000 C CNN
-F 1 "FC-230" H 1450 5400 50  0000 C CNN
-F 2 "Fuse_Holders_and_Fuses:Fuseholder5x20_horiz_open_inline_Type-I" H 1550 5450 60  0001 C CNN
-F 3 "" H 1550 5450 60  0000 C CNN
-	1    1550 5450
-	1    0    0    -1
-$EndComp
-$Comp
 L Diode_Bridge-RESCUE-IACSense D1
 U 1 1 56C0DEF7
@@
 F 0 "P1" H 1100 1400 50  0000 C CNN
 F 1 "CONN_01X03" V 1200 1200 50  0000 C CNN
-F 2 "" H 1100 1200 60  0001 C CNN
+F 2 "Yame_library:Conn3_Term" H 1100 1200 60  0001 C CNN
 F 3 "" H 1100 1200 60  0000 C CNN
 	1    1100 1200
@@
 F 0 "P2" H 1100 2950 50  0000 C CNN
 F 1 "CONN_01X03" V 1200 2750 50  0000 C CNN
-F 2 "" H 1100 2750 60  0001 C CNN
+F 2 "Yame_library:Conn3_Term" H 1100 2750 60  0001 C CNN
 F 3 "" H 1100 2750 60  0000 C CNN
 	1    1100 2750
@@
 P 1450 2000
 F 0 "R1" V 1530 2000 50  0000 C CNN
-F 1 "0.002" V 1450 2000 50  0000 C CNN
-F 2 "Yame_library:SM0603-MR" V 1380 2000 30  0001 C CNN
+F 1 "LRMAM1206-R002FT5" V 1350 2000 50  0000 C CNN
+F 2 "Yame_library:SM1206-MR" V 1380 2000 30  0001 C CNN
 F 3 "" H 1450 2000 30  0000 C CNN
 	1    1450 2000
@@
 P 1950 1400
 F 0 "FB3" H 1950 1550 50  0000 C CNN
-F 1 "LI0805H151R-10" H 1950 1300 50  0000 C CNN
-F 2 "Yame_library:SM0805-MR" H 1950 1400 60  0001 C CNN
+F 1 "BLM18AG102SN1D" H 1950 1300 50  0000 C CNN
+F 2 "Yame_library:SM0603-MR" H 1950 1400 60  0001 C CNN
 F 3 "" H 1950 1400 60  0000 C CNN
 	1    1950 1400
@@
 P 1950 2400
 F 0 "FB4" H 1950 2550 50  0000 C CNN
-F 1 "LI0805H151R-10" H 1950 2300 50  0000 C CNN
-F 2 "Yame_library:SM0805-MR" H 1950 2400 60  0001 C CNN
+F 1 "BLM18AG102SN1D" H 1950 2300 50  0000 C CNN
+F 2 "Yame_library:SM0603-MR" H 1950 2400 60  0001 C CNN
 F 3 "" H 1950 2400 60  0000 C CNN
 	1    1950 2400
@@
 P 1300 4650
 F 0 "FB1" H 1300 4800 50  0000 C CNN
-F 1 "LI0805H151R-10" H 1300 4550 50  0000 C CNN
-F 2 "Yame_library:SM0805-MR" H 1300 4650 60  0001 C CNN
+F 1 "BLM18AG102SN1D" H 1300 4550 50  0000 C CNN
+F 2 "Yame_library:SM0603-MR" H 1300 4650 60  0001 C CNN
 F 3 "" H 1300 4650 60  0000 C CNN
 	1    1300 4650
@@
 P 1400 6350
 F 0 "FB2" H 1400 6500 50  0000 C CNN
-F 1 "LI0805H151R-10" H 1400 6250 50  0000 C CNN
-F 2 "Yame_library:SM0805-MR" H 1400 6350 60  0001 C CNN
+F 1 "BLM18AG102SN1D" H 1400 6250 50  0000 C CNN
+F 2 "Yame_library:SM0603-MR" H 1400 6350 60  0001 C CNN
 F 3 "" H 1400 6350 60  0000 C CNN
 	1    1400 6350
@@
 	1750 6350 2150 6350
 Wire Wire Line
-	1300 5000 1300 5450
+	1300 5000 1300 5550
 Wire Wire Line
 	1300 4200 1300 4300
@@
 	5000 5450 5000 6350
 Wire Wire Line
-	1800 5450 5000 5450
+	1850 5450 5000 5450
 Connection ~ 5450 5650
 Wire Wire Line
@@
 Wire Wire Line
 	10400 1050 10400 1150
+$Comp
+L FUSE_CLIP_5x20 F1
+U 1 1 57424BF5
+P 1600 5450
+F 0 "F1" H 1700 5500 50  0000 C CNN
+F 1 "0751.0062" H 1600 5300 50  0000 C CNN
+F 2 "Yame_library:Fuse_5x20" H 1600 5450 50  0001 C CNN
+F 3 "" H 1600 5450 50  0000 C CNN
+	1    1600 5450
+	1    0    0    -1
+$EndComp
+Wire Wire Line
+	1300 5550 1350 5550
+Wire Wire Line
+	1350 5450 1300 5450
+Connection ~ 1300 5450
+Wire Wire Line
+	1850 5350 1900 5350
+Wire Wire Line
+	1900 5350 1900 5450
+Connection ~ 1900 5450
 $EndSCHEMATC

Commit message: Update IACSense
Parts:
- U3: footprint TO_SOT_Packages_THT:TO-220_Neutral123_Vertical -> Yame_library:SOT23-MR
Changed lines of the file:
@@
 F 0 "U3" H 7150 5900 60  0000 C CNN
 F 1 "MCP1754" H 7600 5450 60  0000 C CNN
-F 2 "TO_SOT_Packages_THT:TO-220_Neutral123_Vertical" H 7350 5700 60  0001 C CNN
+F 2 "Yame_library:SOT23-MR" H 7350 5700 60  0001 C CNN
 F 3 "" H 7350 5700 60  0000 C CNN
 	1    7350 5700

Commit message: update IACSense
Parts:
- P1: value CONN_01X03 -> IN
- P2: value CONN_01X03 -> OUT
- P6: footprint Yame_library:HE10_14-2x4C-2.54-MR -> Yame_library:NRF24L01+
Changed lines of the file:
@@
 F 0 "P6" H 10100 4650 50  0000 C CNN
 F 1 "nRF24L01+" H 10100 4150 50  0000 C CNN
-F 2 "Yame_library:HE10_14-2x4C-2.54-MR" H 10100 3200 50  0001 C CNN
+F 2 "Yame_library:NRF24L01+" H 10100 3200 50  0001 C CNN
 F 3 "" H 10100 3200 50  0000 C CNN
 	1    10100 4400
@@
 P 1100 1200
 F 0 "P1" H 1100 1400 50  0000 C CNN
-F 1 "CONN_01X03" V 1200 1200 50  0000 C CNN
+F 1 "IN" V 1200 1200 50  0000 C CNN
 F 2 "Yame_library:Conn3_Term" H 1100 1200 60  0001 C CNN
 F 3 "" H 1100 1200 60  0000 C CNN
@@
 P 1100 2750
 F 0 "P2" H 1100 2950 50  0000 C CNN
-F 1 "CONN_01X03" V 1200 2750 50  0000 C CNN
+F 1 "OUT" V 1200 2750 50  0000 C CNN
 F 2 "Yame_library:Conn3_Term" H 1100 2750 60  0001 C CNN
 F 3 "" H 1100 2750 60  0000 C CNN
@@
 Text Label 1100 1750 0    60   ~ 0
 Line
-Text Label 1450 1750 0    60   ~ 0
+Text Label 1250 1400 0    60   ~ 0
 Neutral
 Text Label 1400 4200 0    60   ~ 0
 Line
-Text Label 600  6300 0    60   ~ 0
+Text Label 600  6350 0    60   ~ 0
 Neutral
 $Comp
