File: IACSense/IACSense.sch (KiCad schematic (older format))
At the start: 84 parts, among them P1 IN, P2 OUT, P3 zcd, P4 event, P5 Prog, P6 +3.3v, P7 I2C, P8 Test, SW1 SW_Push, U1 MCP39F521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

Commit message: Update IACSense
Parts:
- removed C10: 100n, Capacitors_THT:C_Rect_L16.5mm_W10.7mm_P15.00mm_MKT, symbol C
- added R15, R16: R, Yame_library:SM0201-MR, symbol R
- C3: footprint Capacitors_THT:C_Rect_L11.0mm_W4.2mm_P10.00mm_MKT -> Capacitors_THT:C_Rect_L13.0mm_W6.0mm_P10.00mm_FKS3_FKP3_MKS4
Connections:
- wire segments 236 -> 235
Changed lines of the file:
@@
 Text Label 6850 2350 0    60   ~ 0
 SDA
-Text Label 9000 2100 0    60   ~ 0
+Text Label 8550 2100 0    60   ~ 0
 SCL
-Text Label 9000 2500 0    60   ~ 0
+Text Label 8550 2500 0    60   ~ 0
 SDA
 $Comp
@@
 	10000 1050 10000 1250
 Wire Wire Line
-	9000 2100 9350 2100
+	8550 2100 9000 2100
 Wire Wire Line
 	14950 5950 14950 6050
@@
 	8600 4150 8650 4150
 Wire Wire Line
-	9350 2500 9000 2500
+	8550 2500 9000 2500
 Wire Wire Line
 	10200 5350 10650 5350
@@
 	1    0    0    -1
 $EndComp
-$Comp
-L C C10
-U 1 1 59DE78F2
-P 1900 4600
-F 0 "C10" H 1925 4700 50  0000 L CNN
-F 1 "100n" H 1925 4500 50  0000 L CNN
-F 2 "Capacitors_THT:C_Rect_L16.5mm_W10.7mm_P15.00mm_MKT" H 1938 4450 50  0001 C CNN
-F 3 "" H 1900 4600 50  0001 C CNN
-	1    1900 4600
-	1    0    0    -1
-$EndComp
-Wire Wire Line
-	1900 4250 1900 4450
-Connection ~ 1900 4250
-Wire Wire Line
-	1900 4750 1900 4900
-Wire Wire Line
-	1900 4900 2600 4900
+Wire Wire Line
+	1600 4900 2600 4900
 Wire Wire Line
 	2600 4750 2600 5300
@@
 F 0 "C3" H 1625 4700 50  0000 L CNN
 F 1 "100n" H 1625 4500 50  0000 L CNN
-F 2 "Capacitors_THT:C_Rect_L11.0mm_W4.2mm_P10.00mm_MKT" H 1638 4450 50  0001 C CNN
+F 2 "Capacitors_THT:C_Rect_L13.0mm_W6.0mm_P10.00mm_FKS3_FKP3_MKS4" H 1638 4450 50  0001 C CNN
 F 3 "" H 1600 4600 50  0001 C CNN
 	1    1600 4600
@@
 	1600 4250 1600 4450
 Wire Wire Line
-	1600 4750 1600 4850
-Wire Wire Line
-	1600 4850 1900 4850
-Connection ~ 1900 4850
+	1600 4750 1600 4900
 Text Label 7150 3100 0    60   ~ 0
 ZCD
@@
 	0    1    -1   0
 $EndComp
+$Comp
+L R R16
+U 1 1 59E5209E
+P 9150 2500
+F 0 "R16" V 9230 2500 50  0000 C CNN
+F 1 "R" V 9150 2500 50  0000 C CNN
+F 2 "Yame_library:SM0201-MR" V 9080 2500 50  0001 C CNN
+F 3 "" H 9150 2500 50  0001 C CNN
+	1    9150 2500
+	0    1    1    0
+$EndComp
+$Comp
+L R R15
+U 1 1 59E522A4
+P 9150 2100
+F 0 "R15" V 9230 2100 50  0000 C CNN
+F 1 "R" V 9150 2100 50  0000 C CNN
+F 2 "Yame_library:SM0201-MR" V 9080 2100 50  0001 C CNN
+F 3 "" H 9150 2100 50  0001 C CNN
+	1    9150 2100
+	0    1    1    0
+$EndComp
+Wire Wire Line
+	9300 2100 9350 2100
+Wire Wire Line
+	9300 2500 9350 2500
 $EndSCHEMATC

Commit message: Finish IACSense PCB
Parts:
- added P?: Test, Pin_Headers:Pin_Header_Straight_1x01_Pitch1.00mm, symbol CONN_01X01
Changed lines of the file:
@@
 Text Label 1950 3300 0    60   ~ 0
 Neutral
-Text Label 10750 1700 0    60   ~ 0
-Vtemp
 $Comp
 L FILTER FB6
@@
 	7550 2350 7550 2000
 Wire Wire Line
-	10700 1700 10950 1700
-Wire Wire Line
 	10700 1900 10950 1900
 Wire Wire Line
@@
 Wire Wire Line
 	9300 2500 9350 2500
+$Comp
+L CONN_01X01 P?
+U 1 1 59E6384E
+P 11150 1700
+F 0 "P?" H 11150 1800 50  0000 C CNN
+F 1 "Test" V 11250 1700 50  0000 C CNN
+F 2 "Pin_Headers:Pin_Header_Straight_1x01_Pitch1.00mm" H 11150 1700 60  0001 C CNN
+F 3 "" H 11150 1700 60  0000 C CNN
+	1    11150 1700
+	1    0    0    -1
+$EndComp
+Wire Wire Line
+	10700 1700 10950 1700
 $EndSCHEMATC
