File: IACSense/IACSense.kicad_pcb (KiCad board)
At the start: 2 copper layers, 56.6 x 87.4 mm, 85 parts, among them P1 IN, P2 OUT, P3 zcd, P4 event, P5 Prog, P6 +3.3v, P7 I2C, P8 Test, SW1 SW_Push, U1 MCP39F521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

Commit message: Finish IACSense PCB
Parts:
- added P9: Test, Pin_Headers:Pin_Header_Straight_1x01_Pitch1.00mm, F.Cu at (223.1, 86.5)
- P7: footprint Pin_Headers:Pin_Header_Straight_1x04_Pitch1.00mm -> Pin_Headers:Pin_Header_Straight_1x04_Pitch1.27mm
- R20, R8: moved to F.Cu
- moved FB5 30.2 mm to (194.0, 73.2)
- moved R4 30.2 mm to (196.9, 73.2)
- moved R7 30.1 mm to (199.8, 73.2)
- moved R1 13.0 mm to (197.7, 80.8)
- moved P4 10.9 mm to (227.6, 78.3)
- moved R13 6.95 mm to (220.0, 79.4), turned to 90 degrees
- moved P5 6.62 mm to (230.8, 89.2)
- moved R15 4.89 mm to (224.8, 85.0), turned to 270 degrees
- moved P7 4.06 mm to (218.2, 80.1), turned to 180 degrees
- moved R14 3.65 mm to (216.3, 79.4), turned to 90 degrees
- moved P6 2.75 mm to (232.9, 82.3)
- moved P3 2.16 mm to (221.3, 82.6)
- moved P8 2.15 mm to (221.3, 84.2)
- moved R16 0.81 mm to (225.4, 78.6), turned to 90 degrees
- moved R11 0.45 mm to (198.1, 79.3)
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Connections:
- U4 pad 9: /Vtemp -> Net-(P9-Pad1)
Routing:
- net GND: track 33.9 -> 257.6 mm, vias 2 -> 32
- net /3.3D: track 4.25 -> 134.5 mm, vias 1 -> 5
- net /Tx_BL: track 0.00 -> 57.1 mm, vias 0 -> 1
- net /SCL: track 0.00 -> 56.7 mm, vias 0 -> 1
- net /SDA: track 0.00 -> 52.4 mm, vias 0 -> 3
- net /Rx_BL: track 0.00 -> 49.9 mm, vias 0 -> 1
- net /Line_Out: track 0.00 -> 41.4 mm
- net Net-(P5-Pad4): track 0.00 -> 38.5 mm
- net /Event: track 0.14 -> 36.4 mm, vias 0 -> 2
- net /Neutral: track 76.3 -> 111.7 mm, vias 0 -> 1
- net /Out_SW: track 0.00 -> 25.7 mm, vias 0 -> 2
- net /ZCD: track 0.00 -> 25.5 mm, vias 0 -> 2
- net /3.3A: track 0.00 -> 23.8 mm, vias 0 -> 4
- net Net-(D1-Pad3): track 0.00 -> 18.3 mm
- net Net-(D3-Pad2): track 0.00 -> 15.7 mm
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- added copper zone on B.Cu, net /Line_Out
- added copper zone on B.Cu, net GND
- added copper zone on F.Cu, net GND
Other:
- board size 56.6 x 87.4 mm -> 56.6 x 68 mm
- net class Default: clearance 0.195 -> 0.16; trace_width 0.25 -> 0.16
- rule trace_clearance: 0.195 -> 0.16
- rule trace_min: 0.2 -> 0.16
