File: 2CV/VariBoost.sch (KiCad schematic (older format))
At the start: 27 parts, among them P1 CONN_2, P2 CONN_2, P3 CONN_2, P4 CONN_2, P5 CONN_2, Q1 2N2222, Q3 2N2222, Q4 IRGB14C40L, SW1 SWITCH_INV_2RT, U1 CD4011

Commit message: Update VariBoost
Parts:
- removed C10, C3, C6: 1u, Capacitors_ThroughHole:C_Rect_L7.5_W6.5_P5, symbol C-RESCUE-VariBoost
- removed C5: 100n, Capacitors_ThroughHole:C_Rect_L7_W2.5_P5, symbol C-RESCUE-VariBoost
- removed D1: 10v_1W, Diodes_ThroughHole:Diode_DO-201AD_Horizontal_RM15, symbol ZENER-RESCUE-VariBoost
- removed D3: 10v_1W, Diodes_ThroughHole:Diode_DO-35_SOD27_Horizontal_RM10, symbol ZENER-RESCUE-VariBoost
- removed L1: INDUCTOR, Choke_Toroid_ThroughHole:Choke_Toroid_8x16mm_Vertical, symbol INDUCTOR
- removed P3, P5: CONN_2, Connect:bornier2, symbol CONN_2
- removed Q1, Q3: 2N2222, Housings_TO-92:TO-92_Inline_Wide, symbol 2N2222
- removed R4, R8: 10k, Resistors_ThroughHole:Resistor_Horizontal_RM10mm, symbol R-RESCUE-VariBoost
- removed R5: R, Resistors_ThroughHole:Resistor_Horizontal_RM10mm, symbol R-RESCUE-VariBoost
- removed R9: 100, Resistors_ThroughHole:Resistor_Horizontal_RM20mm, symbol R-RESCUE-VariBoost
- removed U1: CD4011, Housings_DIP:DIP-14_W7.62mm_LongPads, symbol CD4011
- added C?: 1u, Capacitors_ThroughHole:C_Rect_L7.5_W6.5_P5, symbol C-RESCUE-VariBoost
- added C? (x3): 100n, symbol C
- added D? (x3): LED, symbol LED
- added P? (x2): CONN_2, Connect:bornier2, symbol CONN_2
- added P?: CONN_01X05, symbol CONN_01X05
- added Q? (x2): 2N7002E, symbol N-MOS_SOT23
- added R?: 10k, symbol R
- added U?: 7805, symbol 7805
- added U?: PIC16F18323, symbol PIC16F18323
- C1: value 1u -> 10u
- C2: value 1n -> 330p
Connections:
- net labels added: +12V, +5V
- net labels removed: VCC, Vref
- wire segments 66 -> 79
Other:
- note removed: "Connection potar"
- moved on the sheet: C1

Commit message: Update layout
Parts:
- added P? (x3): test, symbol CONN_01X01
- added P?: CONN_2, Connect:bornier2, symbol CONN_2
- added R? (x3): R, symbol R
- U?: value PIC16F18323 -> PIC16F18323_soic
Connections:
- wire segments 79 -> 99
Other:
- moved on the sheet: D?, P?
Changed lines of the file:
@@
 P 7500 6750
 F 0 "U?" H 7100 7300 60  0000 C CNN
-F 1 "PIC16F18323" H 7950 5700 60  0000 C CNN
+F 1 "PIC16F18323_soic" H 7950 5700 60  0000 C CNN
 F 2 "" H 7550 6750 60  0000 C CNN
 F 3 "" H 7550 6750 60  0000 C CNN
@@
 Wire Wire Line
 	7500 7900 7500 7950
-Text Label 7350 6000 0    60   ~ 0
+Text Label 6150 5650 0    60   ~ 0
 +5V
 Wire Wire Line
 	7500 6100 7500 6000
 Wire Wire Line
-	7500 6000 7350 6000
+	6000 5650 6300 5650
 Wire Wire Line
 	6850 7550 6400 7550
@@
 L LED D?
 U 1 1 56DB83D9
-P 8850 5800
-F 0 "D?" H 8850 5900 50  0000 C CNN
-F 1 "LED" H 8850 5700 50  0000 C CNN
-F 2 "" H 8850 5800 50  0000 C CNN
-F 3 "" H 8850 5800 50  0000 C CNN
-	1    8850 5800
+P 9500 5800
+F 0 "D?" H 9500 5900 50  0000 C CNN
+F 1 "LED" H 9500 5700 50  0000 C CNN
+F 2 "" H 9500 5800 50  0000 C CNN
+F 3 "" H 9500 5800 50  0000 C CNN
+	1    9500 5800
 	-1   0    0    1
 $EndComp
@@
 L LED D?
 U 1 1 56DB86E6
-P 8850 6150
-F 0 "D?" H 8850 6250 50  0000 C CNN
-F 1 "LED" H 8850 6050 50  0000 C CNN
-F 2 "" H 8850 6150 50  0000 C CNN
-F 3 "" H 8850 6150 50  0000 C CNN
-	1    8850 6150
+P 9500 6150
+F 0 "D?" H 9500 6250 50  0000 C CNN
+F 1 "LED" H 9500 6050 50  0000 C CNN
+F 2 "" H 9500 6150 50  0000 C CNN
+F 3 "" H 9500 6150 50  0000 C CNN
+	1    9500 6150
 	-1   0    0    1
 $EndComp
@@
 L LED D?
 U 1 1 56DB874D
-P 8850 6500
-F 0 "D?" H 8850 6600 50  0000 C CNN
-F 1 "LED" H 8850 6400 50  0000 C CNN
-F 2 "" H 8850 6500 50  0000 C CNN
-F 3 "" H 8850 6500 50  0000 C CNN
-	1    8850 6500
-	-1   0    0    1
-$EndComp
-Wire Wire Line
-	8650 5800 8300 5800
+P 9500 6500
+F 0 "D?" H 9500 6600 50  0000 C CNN
+F 1 "LED" H 9500 6400 50  0000 C CNN
+F 2 "" H 9500 6500 50  0000 C CNN
+F 3 "" H 9500 6500 50  0000 C CNN
+	1    9500 6500
+	-1   0    0    1
+$EndComp
+Wire Wire Line
+	8300 5800 8900 5800
 Wire Wire Line
 	8300 5800 8300 6550
@@
 	8400 6750 8400 6150
 Wire Wire Line
-	8400 6150 8650 6150
-Wire Wire Line
-	8650 6500 8500 6500
+	8400 6150 8900 6150
+Wire Wire Line
+	8500 6500 8900 6500
 Wire Wire Line
 	8500 6500 8500 6950
@@
 L GND-RESCUE-VariBoost #PWR?
 U 1 1 56DB8AFD
-P 9150 6650
-F 0 "#PWR?" H 9150 6650 30  0001 C CNN
-F 1 "GND" H 9150 6580 30  0001 C CNN
-F 2 "" H 9150 6650 60  0000 C CNN
-F 3 "" H 9150 6650 60  0000 C CNN
-	1    9150 6650
-	1    0    0    -1
-$EndComp
-Wire Wire Line
-	9050 6500 9150 6500
-Wire Wire Line
-	9150 5800 9150 6650
-Wire Wire Line
-	9050 6150 9150 6150
-Connection ~ 9150 6500
-Wire Wire Line
-	9050 5800 9150 5800
-Connection ~ 9150 6150
+P 9800 6650
+F 0 "#PWR?" H 9800 6650 30  0001 C CNN
+F 1 "GND" H 9800 6580 30  0001 C CNN
+F 2 "" H 9800 6650 60  0000 C CNN
+F 3 "" H 9800 6650 60  0000 C CNN
+	1    9800 6650
+	1    0    0    -1
+$EndComp
+Wire Wire Line
+	9700 6500 9800 6500
+Wire Wire Line
+	9800 5800 9800 6650
+Wire Wire Line
+	9700 6150 9800 6150
+Connection ~ 9800 6500
+Wire Wire Line
+	9700 5800 9800 5800
+Connection ~ 9800 6150
 $Comp
 L CONN_01X05 P?
 U 1 1 56DB94B7
-P 6950 4750
-F 0 "P?" H 6950 5050 50  0000 C CNN
-F 1 "CONN_01X05" V 7050 4750 50  0000 C CNN
-F 2 "" H 6950 4750 50  0000 C CNN
-F 3 "" H 6950 4750 50  0000 C CNN
-	1    6950 4750
-	-1   0    0    1
-$EndComp
+P 5800 5650
+F 0 "P?" H 5800 5950 50  0000 C CNN
+F 1 "CONN_01X05" V 5900 5650 50  0000 C CNN
+F 2 "" H 5800 5650 50  0000 C CNN
+F 3 "" H 5800 5650 50  0000 C CNN
+	1    5800 5650
+	-1   0    0    -1
+$EndComp
+Wire Wire Line
+	6850 6550 6800 6550
+Wire Wire Line
+	6800 6550 6800 5450
+Wire Wire Line
+	6800 5450 6000 5450
+Wire Wire Line
+	6850 6750 6700 6750
+Wire Wire Line
+	6700 6750 6700 5550
+Wire Wire Line
+	6700 5550 6000 5550
+Wire Wire Line
+	6000 5750 6600 5750
+Wire Wire Line
+	6600 5750 6600 7150
+Wire Wire Line
+	6600 7150 6850 7150
+$Comp
+L GND-RESCUE-VariBoost #PWR?
+U 1 1 56DB4AAC
+P 6050 5900
+F 0 "#PWR?" H 6050 5900 30  0001 C CNN
+F 1 "GND" H 6050 5830 30  0001 C CNN
+F 2 "" H 6050 5900 60  0000 C CNN
+F 3 "" H 6050 5900 60  0000 C CNN
+	1    6050 5900
+	1    0    0    -1
+$EndComp
+Wire Wire Line
+	6000 5850 6050 5850
+Wire Wire Line
+	6050 5850 6050 5900
+$Comp
+L CONN_01X01 P?
+U 1 1 56DB513D
+P 6500 7350
+F 0 "P?" H 6500 7450 50  0000 C CNN
+F 1 "test" V 6600 7350 50  0000 C CNN
+F 2 "" H 6500 7350 50  0000 C CNN
+F 3 "" H 6500 7350 50  0000 C CNN
+	1    6500 7350
+	-1   0    0    1
+$EndComp
+$Comp
+L CONN_01X01 P?
+U 1 1 56DB5211
+P 8550 7150
+F 0 "P?" H 8550 7250 50  0000 C CNN
+F 1 "test" V 8650 7150 50  0000 C CNN
+F 2 "" H 8550 7150 50  0000 C CNN
+F 3 "" H 8550 7150 50  0000 C CNN
+	1    8550 7150
+	1    0    0    -1
+$EndComp
+$Comp
+L CONN_01X01 P?
+U 1 1 56DB52FA
+P 8550 7350
+F 0 "P?" H 8550 7450 50  0000 C CNN
+F 1 "test" V 8650 7350 50  0000 C CNN
+F 2 "" H 8550 7350 50  0000 C CNN
+F 3 "" H 8550 7350 50  0000 C CNN
+	1    8550 7350
+	1    0    0    -1
+$EndComp
+Wire Wire Line
+	6700 7350 6850 7350
+Wire Wire Line
+	8200 7350 8350 7350
+Wire Wire Line
+	8350 7150 8200 7150
+Text Label 7350 6000 0    60   ~ 0
++5V
+Wire Wire Line
+	7500 6000 7350 6000
+$Comp
+L R R?
+U 1 1 56DB5CA4
+P 9050 5800
+F 0 "R?" V 9130 5800 50  0000 C CNN
+F 1 "R" V 9050 5800 50  0000 C CNN
+F 2 "" V 8980 5800 50  0000 C CNN
+F 3 "" H 9050 5800 50  0000 C CNN
+	1    9050 5800
+	0    1    1    0
+$EndComp
+$Comp
+L R R?
+U 1 1 56DB5DC1
+P 9050 6150
+F 0 "R?" V 9130 6150 50  0000 C CNN
+F 1 "R" V 9050 6150 50  0000 C CNN
+F 2 "" V 8980 6150 50  0000 C CNN
+F 3 "" H 9050 6150 50  0000 C CNN
+	1    9050 6150
+	0    1    1    0
+$EndComp
+$Comp
+L R R?
+U 1 1 56DB5E43
+P 9050 6500
+F 0 "R?" V 9130 6500 50  0000 C CNN
+F 1 "R" V 9050 6500 50  0000 C CNN
+F 2 "" V 8980 6500 50  0000 C CNN
+F 3 "" H 9050 6500 50  0000 C CNN
+	1    9050 6500
+	0    1    1    0
+$EndComp
+Wire Wire Line
+	9200 6150 9300 6150
+Wire Wire Line
+	9200 5800 9300 5800
+Wire Wire Line
+	9200 6500 9300 6500
+$Comp
+L CONN_2 P?
+U 1 1 56DB69A1
+P 12900 8050
+F 0 "P?" V 12850 8050 40  0000 C CNN
+F 1 "CONN_2" V 12950 8050 40  0000 C CNN
+F 2 "Connect:bornier2" H 12900 8050 60  0001 C CNN
+F 3 "" H 12900 8050 60  0000 C CNN
+	1    12900 8050
+	0    -1   -1   0
+$EndComp
+$Comp
+L GND-RESCUE-VariBoost #PWR?
+U 1 1 56DB69A7
+P 12800 8550
+F 0 "#PWR?" H 12800 8550 30  0001 C CNN
+F 1 "GND" H 12800 8480 30  0001 C CNN
+F 2 "" H 12800 8550 60  0000 C CNN
+F 3 "" H 12800 8550 60  0000 C CNN
+	1    12800 8550
+	1    0    0    -1
+$EndComp
+$Comp
+L GND-RESCUE-VariBoost #PWR?
+U 1 1 56DB69AD
+P 13000 8550
+F 0 "#PWR?" H 13000 8550 30  0001 C CNN
+F 1 "GND" H 13000 8480 30  0001 C CNN
+F 2 "" H 13000 8550 60  0000 C CNN
+F 3 "" H 13000 8550 60  0000 C CNN
+	1    13000 8550
+	1    0    0    -1
+$EndComp
+Wire Wire Line
+	13000 8400 13000 8550
+Wire Wire Line
+	12800 8400 12800 8550
 $EndSCHEMATC

Commit message: Finish Variboost µC and send to seeed
Parts:
- removed U?: 7805, symbol 7805
- added C5: 100n, Yame_library:SM0603-MR, symbol C
- added R4: 100, Yame_library:SM0603-MR, symbol R
- added R?: 10k, Yame_library:SM0603-MR, symbol R
- added U1: 7805_SOT252, TO_SOT_Packages_SMD:TO-252-2Lead, symbol 7805_Yame
- C1: footprint Capacitors_ThroughHole:C_Rect_L7.5_W6.5_P5 -> Yame_library:SM0805-MR
- C2: footprint Capacitors_ThroughHole:C_Rect_L7_W2.5_P5 -> Yame_library:SM0603-MR
- C3: renamed from C?; footprint Capacitors_ThroughHole:C_Rect_L7.5_W6.5_P5 -> Yame_library:SM0603-MR
- C4, C6, C7: renamed from C?; footprint (none) -> Yame_library:SM0603-MR
- D1, D3, D4: renamed from D?; footprint (none) -> Yame_library:SM0603-LED-MR
- D2: footprint Diodes_ThroughHole:Diode_DO-35_SOD27_Horizontal_RM10 -> Diodes_SMD:SOD-123
- P6: renamed from P?; footprint (none) -> Yame_library:HE10_14-5C-2.54-MR
- P7, P8, P9: renamed from P?; footprint (none) -> Yame_library:Test_Point_T_H
- Q1, Q2: renamed from Q?; footprint (none) -> Yame_library:SOT23-MR
- R1, R10, R2: footprint Resistors_ThroughHole:Resistor_Horizontal_RM10mm -> Yame_library:SM0603-MR
- R3, R5, R6, R7: renamed from R?; footprint (none) -> Yame_library:SM0603-MR
- U2: renamed from U?; footprint (none) -> Housings_SOIC:SOIC-14_3.9x8.7mm_Pitch1.27mm
- gave numbers to parts that had none: 3
Connections:
- wire segments 99 -> 106
Other:
- moved on the sheet: P5

Commit message: Update Variboost
Parts:
- gave numbers to parts that had none: 1
Changed lines of the file:
@@
 $EndComp
 $Comp
-L GND-RESCUE-VariBoost #PWR01
+L GND-RESCUE-VariBoost #PWR14
 U 1 1 54138F6E
 P 9600 8450
-F 0 "#PWR01" H 9600 8450 30  0001 C CNN
+F 0 "#PWR14" H 9600 8450 30  0001 C CNN
 F 1 "GND" H 9600 8380 30  0001 C CNN
 F 2 "" H 9600 8450 60  0000 C CNN
@@
 $EndComp
 $Comp
-L GND-RESCUE-VariBoost #PWR02
+L GND-RESCUE-VariBoost #PWR17
 U 1 1 54138F75
 P 10250 8350
-F 0 "#PWR02" H 10250 8350 30  0001 C CNN
+F 0 "#PWR17" H 10250 8350 30  0001 C CNN
 F 1 "GND" H 10250 8280 30  0001 C CNN
 F 2 "" H 10250 8350 60  0000 C CNN
@@
 $EndComp
 $Comp
-L GND-RESCUE-VariBoost #PWR03
+L GND-RESCUE-VariBoost #PWR18
 U 1 1 54138F7C
 P 10700 8000
-F 0 "#PWR03" H 10700 8000 30  0001 C CNN
+F 0 "#PWR18" H 10700 8000 30  0001 C CNN
 F 1 "GND" H 10700 7930 30  0001 C CNN
 F 2 "" H 10700 8000 60  0000 C CNN
@@
 $EndComp
 $Comp
-L GND-RESCUE-VariBoost #PWR04
+L GND-RESCUE-VariBoost #PWR3
 U 1 1 5413962D
 P 3650 6750
-F 0 "#PWR04" H 3650 6750 30  0001 C CNN
+F 0 "#PWR3" H 3650 6750 30  0001 C CNN
 F 1 "GND" H 3650 6680 30  0001 C CNN
 F 2 "" H 3650 6750 60  0000 C CNN
@@
 Connection ~ 4950 8050
 $Comp
-L GND-RESCUE-VariBoost #PWR05
+L GND-RESCUE-VariBoost #PWR6
 U 1 1 56381BE2
 P 4950 8600
-F 0 "#PWR05" H 4950 8600 30  0001 C CNN
+F 0 "#PWR6" H 4950 8600 30  0001 C CNN
 F 1 "GND" H 4950 8530 30  0001 C CNN
 F 2 "" H 4950 8600 60  0000 C CNN
@@
 $EndComp
 $Comp
-L GND-RESCUE-VariBoost #PWR06
+L GND-RESCUE-VariBoost #PWR4
 U 1 1 56DB30FD
 P 4350 6550
-F 0 "#PWR06" H 4350 6550 30  0001 C CNN
+F 0 "#PWR4" H 4350 6550 30  0001 C CNN
 F 1 "GND" H 4350 6480 30  0001 C CNN
 F 2 "" H 4350 6550 60  0000 C CNN
@@
 $EndComp
 $Comp
-L GND-RESCUE-VariBoost #PWR07
+L GND-RESCUE-VariBoost #PWR5
 U 1 1 56DB3270
 P 4900 6750
-F 0 "#PWR07" H 4900 6750 30  0001 C CNN
+F 0 "#PWR5" H 4900 6750 30  0001 C CNN
 F 1 "GND" H 4900 6680 30  0001 C CNN
 F 2 "" H 4900 6750 60  0000 C CNN
@@
 $EndComp
 $Comp
-L GND-RESCUE-VariBoost #PWR08
+L GND-RESCUE-VariBoost #PWR1
 U 1 1 56DB5013
 P 1000 9300
-F 0 "#PWR08" H 1000 9300 30  0001 C CNN
+F 0 "#PWR1" H 1000 9300 30  0001 C CNN
 F 1 "GND" H 1000 9230 30  0001 C CNN
 F 2 "" H 1000 9300 60  0000 C CNN
@@
 $EndComp
 $Comp
-L GND-RESCUE-VariBoost #PWR09
+L GND-RESCUE-VariBoost #PWR2
 U 1 1 56DB50A8
 P 1200 9300
-F 0 "#PWR09" H 1200 9300 30  0001 C CNN
+F 0 "#PWR2" H 1200 9300 30  0001 C CNN
 F 1 "GND" H 1200 9230 30  0001 C CNN
 F 2 "" H 1200 9300 60  0000 C CNN
@@
 	1000 9150 1000 9300
 $Comp
-L GND-RESCUE-VariBoost #PWR010
+L GND-RESCUE-VariBoost #PWR7
 U 1 1 56DB5527
 P 5550 8400
-F 0 "#PWR010" H 5550 8400 30  0001 C CNN
+F 0 "#PWR7" H 5550 8400 30  0001 C CNN
 F 1 "GND" H 5550 8330 30  0001 C CNN
 F 2 "" H 5550 8400 60  0000 C CNN
@@
 $EndComp
 $Comp
-L GND-RESCUE-VariBoost #PWR011
+L GND-RESCUE-VariBoost #PWR9
 U 1 1 56DB6FE6
 P 5900 8900
-F 0 "#PWR011" H 5900 8900 30  0001 C CNN
+F 0 "#PWR9" H 5900 8900 30  0001 C CNN
 F 1 "GND" H 5900 8830 30  0001 C CNN
 F 2 "" H 5900 8900 60  0000 C CNN
@@
 $EndComp
 $Comp
-L GND-RESCUE-VariBoost #PWR012
+L GND-RESCUE-VariBoost #PWR12
 U 1 1 56DB7338
 P 6950 8500
-F 0 "#PWR012" H 6950 8500 30  0001 C CNN
+F 0 "#PWR12" H 6950 8500 30  0001 C CNN
 F 1 "GND" H 6950 8430 30  0001 C CNN
 F 2 "" H 6950 8500 60  0000 C CNN
@@
 $EndComp
 $Comp
-L GND-RESCUE-VariBoost #PWR013
+L GND-RESCUE-VariBoost #PWR16
 U 1 1 56DB74ED
 P 10000 8950
-F 0 "#PWR013" H 10000 8950 30  0001 C CNN
+F 0 "#PWR16" H 10000 8950 30  0001 C CNN
 F 1 "GND" H 10000 8880 30  0001 C CNN
 F 2 "" H 10000 8950 60  0000 C CNN
@@
 	10000 8900 10000 8950
 $Comp
-L GND-RESCUE-VariBoost #PWR014
+L GND-RESCUE-VariBoost #PWR13
 U 1 1 56DB7724
 P 7500 7950
-F 0 "#PWR014" H 7500 7950 30  0001 C CNN
+F 0 "#PWR13" H 7500 7950 30  0001 C CNN
 F 1 "GND" H 7500 7880 30  0001 C CNN
 F 2 "" H 7500 7950 60  0000 C CNN
@@
 $EndComp
 $Comp
-L GND-RESCUE-VariBoost #PWR015
+L GND-RESCUE-VariBoost #PWR8
 U 1 1 56DB80C4
 P 5650 6850
-F 0 "#PWR015" H 5650 6850 30  0001 C CNN
+F 0 "#PWR8" H 5650 6850 30  0001 C CNN
 F 1 "GND" H 5650 6780 30  0001 C CNN
 F 2 "" H 5650 6850 60  0000 C CNN
@@
 	8500 6950 8200 6950
 $Comp
-L GND-RESCUE-VariBoost #PWR016
+L GND-RESCUE-VariBoost #PWR15
 U 1 1 56DB8AFD
 P 9800 6650
-F 0 "#PWR016" H 9800 6650 30  0001 C CNN
+F 0 "#PWR15" H 9800 6650 30  0001 C CNN
 F 1 "GND" H 9800 6580 30  0001 C CNN
 F 2 "" H 9800 6650 60  0000 C CNN
@@
 	6600 7150 6850 7150
 $Comp
-L GND-RESCUE-VariBoost #PWR017
+L GND-RESCUE-VariBoost #PWR10
 U 1 1 56DB4AAC
 P 6050 5900
-F 0 "#PWR017" H 6050 5900 30  0001 C CNN
+F 0 "#PWR10" H 6050 5900 30  0001 C CNN
 F 1 "GND" H 6050 5830 30  0001 C CNN
 F 2 "" H 6050 5900 60  0000 C CNN
@@
 $EndComp
 $Comp
-L GND-RESCUE-VariBoost #PWR018
+L GND-RESCUE-VariBoost #PWR19
 U 1 1 56DB69A7
 P 12800 8550
-F 0 "#PWR018" H 12800 8550 30  0001 C CNN
+F 0 "#PWR19" H 12800 8550 30  0001 C CNN
 F 1 "GND" H 12800 8480 30  0001 C CNN
 F 2 "" H 12800 8550 60  0000 C CNN
@@
 $EndComp
 $Comp
-L GND-RESCUE-VariBoost #PWR019
+L GND-RESCUE-VariBoost #PWR20
 U 1 1 56DB69AD
 P 13000 8550
-F 0 "#PWR019" H 13000 8550 30  0001 C CNN
+F 0 "#PWR20" H 13000 8550 30  0001 C CNN
 F 1 "GND" H 13000 8480 30  0001 C CNN
 F 2 "" H 13000 8550 60  0000 C CNN
@@
 Connection ~ 6300 6550
 $Comp
-L GND-RESCUE-VariBoost #PWR020
+L GND-RESCUE-VariBoost #PWR11
 U 1 1 578772DE
 P 6300 7100
-F 0 "#PWR020" H 6300 7100 30  0001 C CNN
+F 0 "#PWR11" H 6300 7100 30  0001 C CNN
 F 1 "GND" H 6300 7030 30  0001 C CNN
 F 2 "" H 6300 7100 60  0000 C CNN
@@
 Connection ~ 5750 6550
 $Comp
-L R R?
+L R R8
 U 1 1 5787E232
 P 5750 6350
-F 0 "R?" V 5830 6350 50  0000 C CNN
+F 0 "R8" V 5830 6350 50  0000 C CNN
 F 1 "10k" V 5750 6350 50  0000 C CNN
 F 2 "Yame_library:SM0603-MR" V 5680 6350 50  0001 C CNN
