File: DAC_Analog/Filter_Out.sch (KiCad schematic (older format))
At the start: 58 parts, among them U10 OPA627xx, U11 TC595002ECB, U2 OPA627xx, U3 OPA627xx, U4 REG104_DCQ, U5 OPA627xx, U6 TC595002ECB, U7 OPA627xx, U8 OPA627xx, U9 REG104_DCQ

Commit message: Update layout
Connections:
- net labels added: +5V_anlg_L, -5V_anlg_L
Other:
- moved on the sheet: C10, C13, C14, C15, C16, C19, C22, C23, C26, C31, C32, C35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
