File: DAC_Analog/DAC_Analog.kicad_pcb (KiCad board)
At the start: 2 copper layers, 100 x 100 mm, 165 parts, among them J1 SPDIF_RX_1, J10 Fix, J11 Fix, J12 Fix, J13 Fix, J14 MCLK_Test, J2 SPDIF_RX_2, J3 SPDIF_RX_3, J4 SPDIF_RX_4, J5 I2C_IN, J6 OutR, J7 OutL, J8 Alim_DAC, J9 Alim_SRC, T1 DA103C, T2 DA103C, T3 DA103C, T4 DA103C, U1 ISO154x, U10 OPA627xx, U11 TC595002ECB, U12 TPS79318, U13 SRC4392, U14 TPS79333, U15 TPS79333, U16 REG104_DCQ, U17 PCM1792A, U18 DS90LV012ATMF, U19 LMK61E2, U2 OPA627xx, U3 OPA627xx, U4 REG104_DCQ, U5 OPA627xx, U6 TC595002ECB, U7 OPA627xx, U8 OPA627xx, U9 REG104_DCQ

Commit message: Update gnd connection on digital transformer
Connections:
- C44 pad 2: Net-(C44-Pad2) -> GND
- C46 pad 2: Net-(C46-Pad2) -> GND
- C48 pad 2: Net-(C48-Pad2) -> GND
- C50 pad 2: Net-(C50-Pad2) -> GND
- R17 pad 2: Net-(C44-Pad2) -> GND
- R18 pad 2: Net-(C46-Pad2) -> GND
- R19 pad 2: Net-(C48-Pad2) -> GND
- R20 pad 2: Net-(C50-Pad2) -> GND
- T1 pad 4: Net-(C44-Pad2) -> GND
- T2 pad 4: Net-(C46-Pad2) -> GND
- T3 pad 4: Net-(C48-Pad2) -> GND
- T4 pad 4: Net-(C50-Pad2) -> GND
Routing:
- net GND: track 1984.2 -> 2000.4 mm
- net Net-(C50-Pad2): track 4.03 -> 0.00 mm
- net Net-(C48-Pad2): track 4.03 -> 0.00 mm
- net Net-(C46-Pad2): track 4.03 -> 0.00 mm
- net Net-(C44-Pad2): track 4.03 -> 0.00 mm
