File: MIG_DF30/MIG_DF30.kicad_pcb (KiCad board)
At the start: 2 copper layers, 159.9 x 99.9 mm, 4 parts

Commit message: Update placing
Parts:
- added A1: Conn_01x01_Male, Yame_library:Pin_d2mm_L11.0mm, F.Cu at (223.5, 63.5)
- added A10: Conn_01x01_Male, Yame_library:Pin_d2mm_L11.0mm, F.Cu at (459.8, 172.4)
- added A11: Conn_01x01_Male, Yame_library:Pin_d2mm_L11.0mm, F.Cu at (173.1, 69.9)
- added A12: Conn_01x01_Male, Yame_library:Pin_d2mm_L11.0mm, F.Cu at (388.0, 98.8)
- added A13: Conn_01x01_Male, Yame_library:Pin_d2mm_L11.0mm, F.Cu at (459.8, 125.9)
- added A14: Conn_01x01_Male, Yame_library:Pin_d2mm_L11.0mm, F.Cu at (417.7, 81.1)
- added A15: Conn_01x01_Male, Yame_library:Pin_d2mm_L11.0mm, F.Cu at (466.5, 169.1)
- added A16: Conn_01x01_Male, Yame_library:FASTON Printed Circuit Board Tabs, F.Cu at (86.6, 67.5)
- added A2: Conn_01x01_Male, Yame_library:Pin_d2mm_L11.0mm, F.Cu at (188.0, 62.1)
- added A3: Conn_01x01_Male, Yame_library:Pin_d2mm_L11.0mm, F.Cu at (196.9, 62.2)
- added A4: Conn_01x01_Male, Yame_library:Pin_d2mm_L11.0mm, F.Cu at (206.9, 62.7)
- added A5: Conn_01x01_Male, Yame_library:Pin_d2mm_L11.0mm, F.Cu at (532.6, 72.8)
- added A6: Conn_01x01_Male, Yame_library:Pin_d2mm_L11.0mm, F.Cu at (519.8, 115.7)
- added A7: Conn_01x01_Male, Yame_library:Pin_d2mm_L11.0mm, F.Cu at (502.3, 130.8)
- added A8: Conn_01x01_Male, Yame_library:Pin_d2mm_L11.0mm, F.Cu at (510.6, 122.7)
- added A9: Conn_01x01_Male, Yame_library:FASTON Printed Circuit Board Tabs, F.Cu at (521.9, 112.1)
- added B1: Conn_01x01_Male, Yame_library:FASTON Printed Circuit Board Tabs, F.Cu at (98.6, 67.5)
- added B2: Conn_01x01_Male, Yame_library:FASTON Printed Circuit Board Tabs, F.Cu at (104.6, 67.5)
- added C1: 0,1u, Yame_library:C_Rect_L24.0mm_W12.2mm_P20mm_MKT, F.Cu at (64.7, 92.2)
- added C10: C, Capacitors_THT:C_Rect_L18.0mm_W6.0mm_P15.00mm_FKS3_FKP3, F.Cu at (402.8, 120.7)
- added C11: C, Capacitors_THT:C_Rect_L18.0mm_W6.0mm_P15.00mm_FKS3_FKP3, F.Cu at (435.4, 105.4)
- added C12: C, Capacitors_THT:C_Rect_L18.0mm_W6.0mm_P15.00mm_FKS3_FKP3, F.Cu at (376.6, 151.3)
- added C13: C, Capacitors_THT:C_Rect_L18.0mm_W7.0mm_P15.00mm_FKS3_FKP3, F.Cu at (446.9, 78.7)
- added C14: C, Capacitors_THT:C_Rect_L13.5mm_W4.0mm_P10.00mm_FKS3_FKP3_MKS4, F.Cu at (395.1, 165.1)
- added C15: CP, Capacitors_THT:CP_Radial_D13.0mm_P5.00mm, F.Cu at (466.3, 123.4)
- added C16: C, Capacitors_THT:C_Rect_L13.5mm_W4.0mm_P10.00mm_FKS3_FKP3_MKS4, F.Cu at (449.8, 118.9)
- added C17: CP, Capacitors_THT:CP_Radial_D13.0mm_P5.00mm, F.Cu at (411.6, 169.6)
- added C18: CP, Capacitors_THT:CP_Radial_D13.0mm_P5.00mm, F.Cu at (431.8, 149.5)
- added C19: CP, Capacitors_THT:CP_Radial_D10.0mm_P5.00mm, F.Cu at (471.5, 142.2)
- added C2: C, Capacitors_THT:C_Rect_L13.5mm_W4.0mm_P10.00mm_FKS3_FKP3_MKS4, F.Cu at (415.3, 154.5)
- added C20: C, Capacitors_THT:C_Rect_L18.0mm_W6.0mm_P15.00mm_FKS3_FKP3, F.Cu at (220.4, 87.2)
- added C21: C, Capacitors_THT:C_Rect_L18.0mm_W6.0mm_P15.00mm_FKS3_FKP3, F.Cu at (231.2, 72.8)
- added C22: C, Capacitors_THT:C_Rect_L18.0mm_W7.0mm_P15.00mm_FKS3_FKP3, F.Cu at (375.9, 144.0)
- added C23: CP, Capacitors_THT:CP_Radial_D8.0mm_P5.00mm, F.Cu at (501.9, 121.1)
- added C24: CP, Capacitors_THT:CP_Radial_D8.0mm_P5.00mm, F.Cu at (481.6, 142.7)
- added C25: C, Capacitors_THT:C_Rect_L13.5mm_W4.0mm_P10.00mm_FKS3_FKP3_MKS4, F.Cu at (490.0, 82.8)
- added C26: C, Capacitors_THT:C_Rect_L13.5mm_W4.0mm_P10.00mm_FKS3_FKP3_MKS4, F.Cu at (475.8, 87.5)
- added C27: C, Capacitors_THT:C_Rect_L18.0mm_W6.0mm_P15.00mm_FKS3_FKP3, F.Cu at (402.8, 114.0)
- added C28: CP, Capacitors_THT:CP_Radial_D8.0mm_P5.00mm, F.Cu at (493.6, 131.3)
- added C29: C, Capacitors_THT:C_Rect_L13.5mm_W4.0mm_P10.00mm_FKS3_FKP3_MKS4, F.Cu at (464.3, 104.7)
- added C3: Conn_01x01_Male, Yame_library:FASTON Printed Circuit Board Tabs, F.Cu at (124.6, 67.4)
- added C30: C, Capacitors_THT:C_Rect_L18.0mm_W6.0mm_P15.00mm_FKS3_FKP3, F.Cu at (384.0, 127.5)
- added C31: CP, Capacitors_THT:CP_Radial_D8.0mm_P5.00mm, F.Cu at (451.1, 176.2)
- added C32: C, Capacitors_THT:C_Rect_L13.5mm_W4.0mm_P10.00mm_FKS3_FKP3_MKS4, F.Cu at (415.3, 145.0)
- added C33: C, Capacitors_THT:C_Rect_L13.5mm_W4.0mm_P10.00mm_FKS3_FKP3_MKS4, F.Cu at (494.0, 76.4)
- added C34: CP, Capacitors_THT:CP_Radial_D8.0mm_P5.00mm, F.Cu at (474.3, 151.9)
- added C35: C, Capacitors_THT:C_Rect_L18.0mm_W6.0mm_P15.00mm_FKS3_FKP3, F.Cu at (357.1, 157.0)
- added C36: C, Capacitors_THT:C_Rect_L18.0mm_W6.0mm_P15.00mm_FKS3_FKP3, F.Cu at (417.7, 88.0)
- added C37: CP, Capacitors_THT:CP_Radial_D8.0mm_P5.00mm, F.Cu at (457.8, 166.2)
- added C38: C, Capacitors_THT:C_Rect_L13.0mm_W4.0mm_P10.00mm_FKS3_FKP3_MKS4, F.Cu at (440.3, 111.2)
- added C39: C, Capacitors_THT:C_Rect_L11.5mm_W5.6mm_P10.00mm_MKT, F.Cu at (502.2, 104.8)
- added C4: C, Capacitors_THT:C_Rect_L18.0mm_W6.0mm_P15.00mm_FKS3_FKP3, F.Cu at (376.6, 158.0)
- added C40: C, Capacitors_THT:C_Rect_L18.0mm_W6.0mm_P15.00mm_FKS3_FKP3, F.Cu at (357.1, 143.5)
- added C41: C, Capacitors_THT:C_Rect_L18.0mm_W6.0mm_P15.00mm_FKS3_FKP3, F.Cu at (357.1, 136.8)
- added C42: C, Capacitors_THT:C_Rect_L18.0mm_W6.0mm_P15.00mm_FKS3_FKP3, F.Cu at (384.0, 120.7)
- added C43: C, Capacitors_THT:C_Rect_L18.0mm_W6.0mm_P15.00mm_FKS3_FKP3, F.Cu at (322.0, 181.5)
- added C44: C, Capacitors_THT:C_Rect_L13.5mm_W4.0mm_P10.00mm_FKS3_FKP3_MKS4, F.Cu at (431.8, 136.1)
- added C45: C, Capacitors_THT:C_Rect_L13.5mm_W4.0mm_P10.00mm_FKS3_FKP3_MKS4, F.Cu at (415.3, 149.8)
- added C46: C, Capacitors_THT:C_Rect_L18.0mm_W6.0mm_P15.00mm_FKS3_FKP3, F.Cu at (375.9, 136.8)
- added C47: C, Capacitors_THT:C_Rect_L13.5mm_W4.0mm_P10.00mm_FKS3_FKP3_MKS4, F.Cu at (464.3, 109.4)
- added C48: C, Capacitors_THT:C_Rect_L13.5mm_W4.0mm_P10.00mm_FKS3_FKP3_MKS4, F.Cu at (445.9, 126.6)
- added C49: C, Capacitors_THT:C_Rect_L13.5mm_W4.0mm_P10.00mm_FKS3_FKP3_MKS4, F.Cu at (431.6, 126.6)
- added C5: C, Capacitors_THT:C_Rect_L18.0mm_W6.0mm_P15.00mm_FKS3_FKP3, F.Cu at (394.6, 134.2)
- added C50: C, Capacitors_THT:C_Rect_L7.2mm_W5.5mm_P5.00mm_FKS2_FKP2_MKS2_MKP2, F.Cu at (383.6, 107.3)
- added C51: CP, Capacitors_THT:CP_Radial_D8.0mm_P5.00mm, F.Cu at (377.3, 89.3)
- added C52: CP, Capacitors_THT:CP_Radial_D8.0mm_P5.00mm, F.Cu at (386.5, 89.3)
- added C53: C, Capacitors_THT:C_Rect_L13.5mm_W4.0mm_P10.00mm_FKS3_FKP3_MKS4, F.Cu at (494.0, 71.7)
- added C54: C, Capacitors_THT:C_Rect_L18.0mm_W8.0mm_P15.00mm_FKS3_FKP3, F.Cu at (345.7, 175.4)
- added C55: C, Capacitors_THT:C_Rect_L13.5mm_W4.0mm_P10.00mm_FKS3_FKP3_MKS4, F.Cu at (415.3, 159.3)
- added C57: CP, Capacitors_THT:CP_Radial_D8.0mm_P5.00mm, F.Cu at (465.2, 155.9)
- added C58: CP, Capacitors_THT:CP_Radial_D8.0mm_P5.00mm, F.Cu at (503.4, 112.3)
- added C59: C, Capacitors_THT:C_Rect_L13.5mm_W4.0mm_P10.00mm_FKS3_FKP3_MKS4, F.Cu at (477.6, 92.3)
- added C6: C, Capacitors_THT:C_Rect_L18.0mm_W8.0mm_P15.00mm_FKS3_FKP3, F.Cu at (112.1, 78.9)
- added C60: C, Capacitors_THT:C_Rect_L13.5mm_W4.0mm_P10.00mm_FKS3_FKP3_MKS4, F.Cu at (431.6, 131.4)
- added C61: C, Capacitors_THT:C_Rect_L13.5mm_W4.0mm_P10.00mm_FKS3_FKP3_MKS4, F.Cu at (475.8, 82.8)
- added C62: C, Capacitors_THT:C_Rect_L18.0mm_W6.0mm_P15.00mm_FKS3_FKP3, F.Cu at (384.0, 114.0)
- added C63: CP, Capacitors_THT:CP_Radial_D8.0mm_P5.00mm, F.Cu at (441.9, 177.0)
- added C64: C, Capacitors_THT:C_Rect_L13.5mm_W4.0mm_P10.00mm_FKS3_FKP3_MKS4, F.Cu at (377.4, 182.1)
- added C65: CP, Capacitors_THT:CP_Radial_D8.0mm_P5.00mm, F.Cu at (515.6, 106.0)
- added C66: CP, Capacitors_THT:CP_Radial_D8.0mm_P5.00mm, F.Cu at (526.1, 95.7)
- added C67: C, Capacitors_THT:C_Rect_L18.0mm_W6.0mm_P15.00mm_FKS3_FKP3, F.Cu at (357.1, 150.3)
- added C68: C, Capacitors_THT:C_Rect_L18.0mm_W6.0mm_P15.00mm_FKS3_FKP3, F.Cu at (421.5, 112.2)
- added C69: C, Capacitors_THT:C_Rect_L18.0mm_W6.0mm_P15.00mm_FKS3_FKP3, F.Cu at (394.6, 141.0)
- added C7: C, Capacitors_THT:C_Rect_L13.5mm_W4.0mm_P10.00mm_FKS3_FKP3_MKS4, F.Cu at (464.3, 99.9)
- added C70: C, Capacitors_THT:C_Rect_L18.0mm_W6.0mm_P15.00mm_FKS3_FKP3, F.Cu at (402.8, 127.5)
- added C8: C, Capacitors_THT:C_Rect_L18.0mm_W6.0mm_P15.00mm_FKS3_FKP3, F.Cu at (470.7, 68.3)
- added C9: C, Capacitors_THT:C_Rect_L18.0mm_W6.0mm_P15.00mm_FKS3_FKP3, F.Cu at (440.4, 94.8)
- added D1: Conn_01x01_Male, Yame_library:FASTON Printed Circuit Board Tabs, F.Cu at (74.1, 67.4)
- added D10: D, Diodes_THT:D_DO-15_P10.16mm_Horizontal, F.Cu at (247.0, 82.1)
- added D11: D, Diodes_THT:D_DO-35_SOD27_P10.16mm_Horizontal, F.Cu at (445.0, 137.1)
- added D12: D, Diodes_THT:D_DO-35_SOD27_P10.16mm_Horizontal, F.Cu at (477.5, 102.0)
- added D13: D, Diodes_THT:D_DO-35_SOD27_P10.16mm_Horizontal, F.Cu at (448.8, 122.7)
- added D14: D, Diodes_THT:D_DO-41_SOD81_P10.16mm_Horizontal, F.Cu at (431.1, 140.2)
- added D15: D, Diodes_THT:D_DO-41_SOD81_P10.16mm_Horizontal, F.Cu at (439.9, 99.9)
- added D16: D, Diodes_THT:D_DO-35_SOD27_P10.16mm_Horizontal, F.Cu at (507.2, 76.2)
- added D17: D, Diodes_THT:D_DO-35_SOD27_P10.16mm_Horizontal, F.Cu at (507.2, 73.4)
- added D18: D, Diodes_THT:D_DO-35_SOD27_P10.16mm_Horizontal, F.Cu at (477.5, 104.8)
- added D19: D_Bridge_+A-A, Diodes_THT:Diode_Bridge_Round_D9.8mm, F.Cu at (455.2, 154.1)
- added D2: D, Yame_library:D_P600_R-6_P18.00mm_Horizontal, F.Cu at (76.6, 94.9)
- added D20: D, Diodes_THT:D_DO-35_SOD27_P10.16mm_Horizontal, F.Cu at (507.2, 70.7)
- added D21: D, Diodes_THT:D_DO-35_SOD27_P10.16mm_Horizontal, F.Cu at (476.6, 96.0)
- added D22: D, Diodes_THT:D_DO-41_SOD81_P10.16mm_Horizontal, F.Cu at (489.3, 86.9)
- added D23: D, Diodes_THT:D_DO-41_SOD81_P10.16mm_Horizontal, F.Cu at (445.1, 130.7)
- added D24: D, Diodes_THT:D_DO-35_SOD27_P10.16mm_Horizontal, F.Cu at (403.7, 183.9)
- added D25: D, Diodes_THT:D_DO-35_SOD27_P10.16mm_Horizontal, F.Cu at (422.0, 163.0)
- added D26: D, Diodes_THT:D_DO-35_SOD27_P10.16mm_Horizontal, F.Cu at (520.0, 66.3)
- added D27: D, Diodes_THT:D_DO-35_SOD27_P10.16mm_Horizontal, F.Cu at (503.2, 83.4)
- added D28: D, Diodes_THT:D_DO-35_SOD27_P10.16mm_Horizontal, F.Cu at (428.5, 157.8)
- added D29: D, Diodes_THT:D_DO-35_SOD27_P10.16mm_Horizontal, F.Cu at (477.5, 107.5)
- added D3: D, Yame_library:D_P600_R-6_P18.00mm_Horizontal, F.Cu at (89.6, 94.9)
- added D30: D, Diodes_THT:D_DO-35_SOD27_P10.16mm_Horizontal, F.Cu at (403.7, 181.1)
- added D4: D, Yame_library:D_P600_R-6_P18.00mm_Horizontal, F.Cu at (102.1, 94.9)
- added D5: D, Yame_library:D_P600_R-6_P18.00mm_Horizontal, F.Cu at (123.6, 94.9)
- added D6: D, Yame_library:D_P600_R-6_P18.00mm_Horizontal, F.Cu at (136.1, 94.9)
- added D7: D, Yame_library:D_P600_R-6_P18.00mm_Horizontal, F.Cu at (184.1, 90.9)
- added D8: D_Bridge_+A-A, Diodes_THT:Diode_Bridge_Round_D9.8mm, F.Cu at (516.1, 93.9)
- added D9: D, Diodes_THT:D_DO-15_P10.16mm_Horizontal, F.Cu at (240.8, 82.0)
- added E1: Conn_01x01_Male, Yame_library:FASTON Printed Circuit Board Tabs, F.Cu at (159.1, 67.5)
- added E2: Conn_01x01_Male, Yame_library:FASTON Printed Circuit Board Tabs, F.Cu at (165.6, 67.5)
- added F1: Conn_01x01_Male, Yame_library:FASTON Printed Circuit Board Tabs, F.Cu at (179.6, 67.5)
- added G1: Conn_01x01_Male, Yame_library:FASTON Printed Circuit Board Tabs, F.Cu at (139.1, 67.5)
- added G2: Conn_01x01_Male, Yame_library:FASTON Printed Circuit Board Tabs, F.Cu at (149.1, 67.5)
- added H1: MountingHole_Pad, Yame_library:MountingHole_5.5mm_Square_Pad, F.Cu at (61.1, 101.4)
- added H2: Conn_01x01_Male, Yame_library:Pin_d2mm_L11.0mm, F.Cu at (65.1, 65.9)
- added K1: G5V-2, Yame_library:Relay_DPDT_1, F.Cu at (371.8, 106.9)
- added K2: G5V-2, Yame_library:Relay_DPDT_1, F.Cu at (358.3, 106.9)
- added Q1: TIC116, Yame_library:TO-220-3_Horizontal_1, F.Cu at (337.7, 95.5)
- added Q10: Q_NJFET_SGD, TO_SOT_Packages_THT:TO-18-3, F.Cu at (424.1, 148.5)
- added Q11: BC107, TO_SOT_Packages_THT:TO-18-3, F.Cu at (424.1, 155.2)
- added Q12: 2N3905, TO_SOT_Packages_THT:TO-18-3, F.Cu at (430.8, 148.5)
- added Q13: BC107, TO_SOT_Packages_THT:TO-18-3, F.Cu at (430.8, 155.2)
- added Q14: BC107, TO_SOT_Packages_THT:TO-18-3, F.Cu at (437.5, 148.5)
- added Q2: TIC116, Yame_library:TO-220-3_Horizontal_1, F.Cu at (337.7, 127.6)
- added Q3: TIC116, Yame_library:TO-220-3_Horizontal_1, F.Cu at (337.7, 159.6)
- added Q5: 2N3905, TO_SOT_Packages_THT:TO-39-3, F.Cu at (448.1, 166.8)
- added Q6: BC107, TO_SOT_Packages_THT:TO-18-3, F.Cu at (310.1, 109.9)
- added Q7: BC107, TO_SOT_Packages_THT:TO-18-3, F.Cu at (417.4, 148.5)
- added Q8: 2N3905, TO_SOT_Packages_THT:TO-39-3, F.Cu at (483.9, 133.4)
- added Q9: BC107, TO_SOT_Packages_THT:TO-18-3, F.Cu at (417.4, 155.2)
- added R1: R, Resistors_THT:R_Axial_DIN0207_L6.3mm_D2.5mm_P10.16mm_Horizontal, F.Cu at (503.2, 80.4)
- added R10: R, Resistors_THT:R_Axial_Power_L25.0mm_W6.4mm_P27.94mm, F.Cu at (391.9, 68.5)
- added R11: R, Resistors_THT:R_Axial_Power_L25.0mm_W6.4mm_P27.94mm, F.Cu at (321.6, 164.7)
- added R12: R, Resistors_THT:R_Axial_Power_L25.0mm_W6.4mm_P27.94mm, F.Cu at (391.9, 75.7)
- added R13: R, Resistors_THT:R_Axial_DIN0207_L6.3mm_D2.5mm_P10.16mm_Horizontal, F.Cu at (416.1, 178.1)
- added R14: R, Resistors_THT:R_Axial_DIN0207_L6.3mm_D2.5mm_P10.16mm_Horizontal, F.Cu at (457.4, 135.2)
- added R15: R, Resistors_THT:R_Axial_DIN0207_L6.3mm_D2.5mm_P10.16mm_Horizontal, F.Cu at (442.3, 150.1)
- added R16: R, Resistors_THT:R_Axial_DIN0207_L6.3mm_D2.5mm_P10.16mm_Horizontal, F.Cu at (422.0, 169.3)
- added R17: R, Resistors_THT:R_Axial_DIN0411_L9.9mm_D3.6mm_P15.24mm_Horizontal, F.Cu at (489.0, 67.1)
- added R18: R, Resistors_THT:R_Axial_DIN0207_L6.3mm_D2.5mm_P10.16mm_Horizontal, F.Cu at (519.5, 72.6)
- added R19: R, Resistors_THT:R_Axial_DIN0207_L6.3mm_D2.5mm_P10.16mm_Horizontal, F.Cu at (475.6, 113.8)
- added R2: R, Resistors_THT:R_Axial_DIN0207_L6.3mm_D2.5mm_P10.16mm_Horizontal, F.Cu at (490.8, 93.5)
- added R20: R, Resistors_THT:R_Axial_DIN0207_L6.3mm_D2.5mm_P10.16mm_Horizontal, F.Cu at (489.8, 100.0)
- added R21: R, Resistors_THT:R_Axial_DIN0207_L6.3mm_D2.5mm_P10.16mm_Horizontal, F.Cu at (503.2, 89.7)
- added R22: R, Resistors_THT:R_Axial_DIN0207_L6.3mm_D2.5mm_P10.16mm_Horizontal, F.Cu at (489.8, 96.7)
- added R23: R, Resistors_THT:R_Axial_DIN0207_L6.3mm_D2.5mm_P10.16mm_Horizontal, F.Cu at (477.5, 110.5)
- added R24: R, Resistors_THT:R_Axial_DIN0207_L6.3mm_D2.5mm_P10.16mm_Horizontal, F.Cu at (443.7, 140.1)
- added R25: R, Resistors_THT:R_Axial_DIN0207_L6.3mm_D2.5mm_P10.16mm_Horizontal, F.Cu at (520.0, 69.3)
- added R26: R, Resistors_THT:R_Axial_DIN0207_L6.3mm_D2.5mm_P10.16mm_Horizontal, F.Cu at (422.0, 166.0)
- added R27: R, Resistors_THT:R_Axial_DIN0207_L6.3mm_D2.5mm_P10.16mm_Horizontal, F.Cu at (442.3, 146.8)
- added R28: R, Resistors_THT:R_Axial_DIN0207_L6.3mm_D2.5mm_P10.16mm_Horizontal, F.Cu at (457.8, 131.9)
- added R29: R, Resistors_THT:R_Axial_DIN0207_L6.3mm_D2.5mm_P10.16mm_Horizontal, F.Cu at (442.3, 143.6)
- added R3: R, Resistors_THT:R_Axial_DIN0414_L11.9mm_D4.5mm_P5.08mm_Vertical, F.Cu at (112.1, 70.9)
- added R30: R, Resistors_THT:R_Axial_DIN0411_L9.9mm_D3.6mm_P15.24mm_Horizontal, F.Cu at (413.0, 140.5)
- added R31: R, Resistors_THT:R_Axial_DIN0207_L6.3mm_D2.5mm_P10.16mm_Horizontal, F.Cu at (434.4, 161.3)
- added R32: R, Resistors_THT:R_Axial_DIN0207_L6.3mm_D2.5mm_P10.16mm_Horizontal, F.Cu at (515.6, 79.2)
- added R33: R, Resistors_THT:R_Axial_DIN0207_L6.3mm_D2.5mm_P10.16mm_Horizontal, F.Cu at (489.8, 106.5)
- added R34: R, Resistors_THT:R_Axial_DIN0207_L6.3mm_D2.5mm_P10.16mm_Horizontal, F.Cu at (416.1, 181.4)
- added R35: R, Resistors_THT:R_Axial_DIN0207_L6.3mm_D2.5mm_P10.16mm_Horizontal, F.Cu at (476.8, 120.3)
- added R36: R, Resistors_THT:R_Axial_DIN0207_L6.3mm_D2.5mm_P10.16mm_Horizontal, F.Cu at (440.9, 158.0)
- added R37: R, Resistors_THT:R_Axial_DIN0207_L6.3mm_D2.5mm_P10.16mm_Horizontal, F.Cu at (445.0, 134.1)
- added R38: R, Resistors_THT:R_Axial_DIN0207_L6.3mm_D2.5mm_P10.16mm_Horizontal, F.Cu at (515.6, 82.4)
- added R39: R, Resistors_THT:R_Axial_DIN0207_L6.3mm_D2.5mm_P10.16mm_Horizontal, F.Cu at (454.6, 143.4)
- added R4: R, Resistors_THT:R_Axial_DIN0207_L6.3mm_D2.5mm_P10.16mm_Horizontal, F.Cu at (519.5, 75.8)
- added R40: R, Resistors_THT:R_Axial_DIN0207_L6.3mm_D2.5mm_P10.16mm_Horizontal, F.Cu at (457.4, 138.4)
- added R41: R, Resistors_THT:R_Axial_DIN0207_L6.3mm_D2.5mm_P10.16mm_Horizontal, F.Cu at (434.4, 164.5)
- added R42: R, Resistors_THT:R_Axial_DIN0207_L6.3mm_D2.5mm_P10.16mm_Horizontal, F.Cu at (502.2, 96.7)
- added R43: R, Resistors_THT:R_Axial_DIN0207_L6.3mm_D2.5mm_P10.16mm_Horizontal, F.Cu at (470.1, 131.9)
- added R44: R, Resistors_THT:R_Axial_DIN0411_L9.9mm_D3.6mm_P15.24mm_Horizontal, F.Cu at (376.2, 167.9)
- added R45: R, Resistors_THT:R_Axial_DIN0207_L6.3mm_D2.5mm_P10.16mm_Horizontal, F.Cu at (454.6, 146.6)
- added R46: R, Resistors_THT:R_Axial_DIN0411_L9.9mm_D3.6mm_P15.24mm_Horizontal, F.Cu at (475.1, 73.9)
- added R47: R, Resistors_THT:R_Axial_DIN0207_L6.3mm_D2.5mm_P10.16mm_Horizontal, F.Cu at (515.6, 85.7)
- added R48: R, Resistors_THT:R_Axial_DIN0411_L9.9mm_D3.6mm_P15.24mm_Horizontal, F.Cu at (431.0, 117.7)
- added R49: R, Resistors_THT:R_Axial_DIN0207_L6.3mm_D2.5mm_P10.16mm_Horizontal, F.Cu at (476.8, 123.5)
- added R5: R, Resistors_THT:R_Axial_DIN0309_L9.0mm_D3.2mm_P15.24mm_Horizontal, F.Cu at (382.4, 176.4)
- added R50: R, Resistors_THT:R_Axial_DIN0207_L6.3mm_D2.5mm_P10.16mm_Horizontal, F.Cu at (503.2, 86.4)
- added R51: R, Resistors_THT:R_Axial_DIN0411_L9.9mm_D3.6mm_P15.24mm_Horizontal, F.Cu at (431.0, 122.1)
- added R52: R, Resistors_THT:R_Axial_DIN0207_L6.3mm_D2.5mm_P10.16mm_Horizontal, F.Cu at (489.8, 109.7)
- added R53: R, Resistors_THT:R_Axial_DIN0411_L9.9mm_D3.6mm_P15.24mm_Horizontal, F.Cu at (376.2, 163.6)
- added R54: R, Resistors_THT:R_Axial_DIN0207_L6.3mm_D2.5mm_P10.16mm_Horizontal, F.Cu at (477.5, 99.0)
- added R55: R, Resistors_THT:R_Axial_DIN0411_L9.9mm_D3.6mm_P15.24mm_Horizontal, F.Cu at (413.0, 136.1)
- added R56: R, Resistors_THT:R_Axial_DIN0207_L6.3mm_D2.5mm_P10.16mm_Horizontal, F.Cu at (463.2, 113.4)
- added R57: R, Resistors_THT:R_Axial_DIN0411_L9.9mm_D3.6mm_P15.24mm_Horizontal, F.Cu at (358.5, 181.9)
- added R58: R, Resistors_THT:R_Axial_DIN0411_L9.9mm_D3.6mm_P15.24mm_Horizontal, F.Cu at (382.8, 172.3)
- added R59: R, Resistors_THT:R_Axial_DIN0411_L9.9mm_D3.6mm_P15.24mm_Horizontal, F.Cu at (458.8, 95.4)
- added R6: R, Resistors_THT:R_Axial_DIN0207_L6.3mm_D2.5mm_P10.16mm_Horizontal, F.Cu at (476.8, 117.0)
- added R60: R, Resistors_THT:R_Axial_DIN0207_L6.3mm_D2.5mm_P10.16mm_Horizontal, F.Cu at (403.7, 178.1)
- added R61: R, Resistors_THT:R_Axial_DIN0411_L9.9mm_D3.6mm_P15.24mm_Horizontal, F.Cu at (475.1, 78.2)
- added R62: R, Resistors_THT:R_Axial_DIN0207_L6.3mm_D2.5mm_P10.16mm_Horizontal, F.Cu at (503.2, 92.9)
- added R63: R, Resistors_THT:R_Axial_DIN0411_L9.9mm_D3.6mm_P15.24mm_Horizontal, F.Cu at (340.3, 181.9)
- added R64: R, Resistors_THT:R_Axial_DIN0207_L6.3mm_D2.5mm_P10.16mm_Horizontal, F.Cu at (515.5, 89.7)
- added R65: R, Resistors_THT:R_Axial_DIN0207_L6.3mm_D2.5mm_P10.16mm_Horizontal, F.Cu at (476.8, 126.8)
- added R66: R, Resistors_THT:R_Axial_DIN0207_L6.3mm_D2.5mm_P10.16mm_Horizontal, F.Cu at (454.6, 149.9)
- added R67: R, Resistors_THT:R_Axial_DIN0207_L6.3mm_D2.5mm_P10.16mm_Horizontal, F.Cu at (502.2, 100.0)
- added R68: R, Resistors_THT:R_Axial_DIN0207_L6.3mm_D2.5mm_P10.16mm_Horizontal, F.Cu at (434.4, 171.0)
- added R69: R, Resistors_THT:R_Axial_DIN0207_L6.3mm_D2.5mm_P10.16mm_Horizontal, F.Cu at (428.4, 175.8)
- added R7: R, Resistors_THT:R_Axial_DIN0207_L6.3mm_D2.5mm_P10.16mm_Horizontal, F.Cu at (422.0, 172.5)
- added R70: R, Resistors_THT:R_Axial_DIN0207_L6.3mm_D2.5mm_P10.16mm_Horizontal, F.Cu at (469.7, 135.2)
- added R71: R, Resistors_THT:R_Axial_DIN0207_L6.3mm_D2.5mm_P10.16mm_Horizontal, F.Cu at (490.8, 90.2)
- added R72: R, Resistors_THT:R_Axial_DIN0207_L6.3mm_D2.5mm_P10.16mm_Horizontal, F.Cu at (487.9, 113.8)
- added R73: R, Resistors_THT:R_Axial_DIN0207_L6.3mm_D2.5mm_P10.16mm_Horizontal, F.Cu at (434.4, 167.8)
- added R8: R, Resistors_THT:R_Axial_Power_L25.0mm_W6.4mm_P27.94mm, F.Cu at (253.0, 87.5)
- added R88: R, Resistors_THT:R_Axial_DIN0207_L6.3mm_D2.5mm_P10.16mm_Horizontal, F.Cu at (442.3, 153.3)
- added R9: R, Resistors_THT:R_Axial_DIN0207_L6.3mm_D2.5mm_P10.16mm_Horizontal, F.Cu at (489.8, 103.2)
- added RV1: R_POT, Potentiometers:Potentiometer_Trimmer_VishaySpectrol_Econtrim-Type36T, F.Cu at (428.9, 183.9)
- added RV2: R_POT, Potentiometers:Potentiometer_Trimmer_VishaySpectrol_Econtrim-Type36T, F.Cu at (525.4, 106.6)
- added RV3: R_POT, Yame_library:Potentiometer_MIG, F.Cu at (406.6, 101.3)
- added U1: 4001, Housings_DIP:DIP-14_W7.62mm, F.Cu at (404.5, 145.9)
- added U100: LM317_3PinPackage, Yame_library:TO-220-3_Horizontal_1, F.Cu at (372.8, 95.5)
- added U2: 4001, Housings_DIP:DIP-14_W7.62mm, F.Cu at (453.4, 99.7)
- added U3: 4011, Housings_DIP:DIP-14_W7.62mm, F.Cu at (394.6, 145.9)
- added U4: LM324, Housings_DIP:DIP-14_W7.62mm, F.Cu at (376.2, 86.5)
- added U5: LM324, Housings_DIP:DIP-14_W7.62mm, F.Cu at (464.9, 76.4)
- added U6: 4001, Housings_DIP:DIP-14_W7.62mm, F.Cu at (420.8, 117.1)
- added U7: LM2907N, Housings_DIP:DIP-14_W7.62mm, F.Cu at (386.1, 86.5)
- moved MK3 474.2 mm to (529.8, 86.4)
- moved MK1 364.2 mm to (402.5, 170.5)
- moved MK2 319.0 mm to (529.8, 80.4)
- moved MK4 272.1 mm to (484.2, 150.1)
Other:
- board size 159.9 x 99.9 mm -> 200 x 190 mm

Commit message: Finish placing
Parts:
- removed MK1, MK2, MK3, MK4: Mounting_Hole_PAD, Mounting_Holes:MountingHole_2.7mm
- added H3: MountingHole_Pad, Mounting_Holes:MountingHole_5.5mm, F.Cu at (61.1, 238.9)
- A9: footprint Yame_library:FASTON Printed Circuit Board Tabs -> Yame_library:Pin_d2mm_L11.0mm
- C62: footprint Capacitors_THT:C_Rect_L18.0mm_W6.0mm_P15.00mm_FKS3_FKP3 -> Capacitors_THT:C_Rect_L13.5mm_W4.0mm_P10.00mm_FKS3_FKP3_MKS4
- R44, R46, R48, R51, R53, R55, R57, R58, R59, R61, R63: footprint Resistors_THT:R_Axial_DIN0411_L9.9mm_D3.6mm_P15.24mm_Horizontal -> Resistors_THT:R_Axial_DIN0207_L6.3mm_D2.5mm_P10.16mm_Horizontal
- moved R32 458.5 mm to (78.6, 217.9)
- moved R38 429.8 mm to (105.1, 209.8), turned to 270 degrees
- moved Q8 425.7 mm to (64.1, 203.9), turned to 90 degrees
- moved D22 421.0 mm to (95.6, 235.9), turned to 90 degrees
- moved D21 417.8 mm to (78.6, 222.9)
- moved R9 415.2 mm to (80.7, 173.9), turned to 180 degrees
- moved R33 410.0 mm to (93.1, 209.8), turned to 270 degrees
- moved C47 407.3 mm to (65.1, 189.9)
- moved R18 399.8 mm to (125.6, 140.9), turned to 270 degrees
- moved R47 399.1 mm to (136.1, 209.3), turned to 270 degrees
- moved R1 397.6 mm to (106.1, 100.4), turned to 270 degrees
- moved C25 395.3 mm to (104.1, 168.4), turned to 90 degrees
- moved R42 393.1 mm to (125.6, 209.3), turned to 270 degrees
- moved R35 390.6 mm to (96.6, 209.8), turned to 270 degrees
- moved R2 386.3 mm to (107.1, 137.4), turned to 90 degrees
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Connections:
- D18 pad 1: Net-(C13-Pad1) -> Net-(A10-Pad1)
- D18 pad 2: Net-(A10-Pad1) -> Net-(C13-Pad1)
- D2 pad 1: Net-(B1-Pad1) -> Net-(D1-Pad1)
- D2 pad 2: Net-(D1-Pad1) -> Net-(B1-Pad1)
- D26 pad 1: GND -> Net-(C33-Pad2)
- D26 pad 2: Net-(C33-Pad2) -> GND
- D27 pad 1: Net-(C54-Pad2) -> Net-(D27-Pad1)
- D27 pad 2: Net-(D27-Pad2) -> Net-(C54-Pad2)
- D28 pad 1: /-Valim -> Net-(C54-Pad2)
- D28 pad 2: Net-(C54-Pad2) -> /-Valim
- D3 pad 1: Net-(C10-Pad2) -> Net-(B1-Pad1)
- D3 pad 2: Net-(B1-Pad1) -> Net-(C10-Pad2)
- D4 pad 1: Net-(C10-Pad2) -> Net-(B1-Pad1)
- D4 pad 2: Net-(B1-Pad1) -> Net-(C10-Pad2)
- D5 pad 1: Net-(C10-Pad2) -> Net-(C3-Pad1)
- D5 pad 2: Net-(C3-Pad1) -> Net-(C10-Pad2)
- D6 pad 1: Net-(C10-Pad2) -> Net-(C3-Pad1)
- D6 pad 2: Net-(C3-Pad1) -> Net-(C10-Pad2)
- D7 pad 1: Net-(C10-Pad2) -> Net-(C14-Pad2)
- D7 pad 2: Net-(C14-Pad2) -> Net-(C10-Pad2)
- Q10 pad 2: Net-(D25-Pad1) -> Net-(D25-Pad2)
- R34 pad 2: Net-(D25-Pad1) -> Net-(D25-Pad2)
- R40 pad 1: Net-(Q12-Pad2) -> Net-(Q12-Pad1)
- R61 pad 2: Net-(D27-Pad2) -> Net-(D27-Pad1)
- RV1 pad 1: Net-(R7-Pad2) -> GND
- RV1 pad 3: GND -> Net-(R7-Pad2)
- RV3 pad 1: Net-(C36-Pad1) -> Net-(D16-Pad2)
- RV3 pad 3: Net-(D16-Pad2) -> Net-(C36-Pad1)
- U5 pad 1: Net-(D25-Pad2) -> Net-(D25-Pad1)
- U5 pad 10: Net-(D27-Pad2) -> Net-(D27-Pad1)

Commit message: Start layout
Parts:
- moved C1 21.3 mm to (63.6, 70.9), turned to 270 degrees
- moved D18 10.2 mm to (203.1, 160.9), turned to 180 degrees
- moved R26 10.2 mm to (203.1, 164.4), turned to 180 degrees
- moved R88 10.2 mm to (132.1, 226.9), turned to 270 degrees
- moved R39 10.1 mm to (109.7, 209.8), turned to 270 degrees
- moved C50 4.83 mm to (89.9, 235.4), turned to 180 degrees
- moved R8 2.00 mm to (251.6, 91.4)
- moved RV1 0.91 mm to (247.2, 118.0)
Connections:
- C28 pad 1: Net-(C28-Pad1) -> /A1
- C31 pad 1: Net-(C28-Pad1) -> /A1
- C35 pad 1: Net-(C28-Pad1) -> /A1
- C37 pad 1: Net-(C28-Pad1) -> /A1
- C52 pad 1: Net-(C28-Pad1) -> /A1
- C63 pad 1: Net-(C28-Pad1) -> /A1
- D11 pad 2: Net-(D11-Pad2) -> GND
- D12 pad 1: Net-(D11-Pad2) -> GND
- D14 pad 1: Net-(D14-Pad1) -> /Q3_G
- D14 pad 2: /Q3_G -> Net-(D14-Pad2)
- D2 pad 1: Net-(D1-Pad1) -> Net-(B1-Pad1)
- D2 pad 2: Net-(B1-Pad1) -> Net-(D1-Pad1)
- D3 pad 1: Net-(B1-Pad1) -> Net-(C10-Pad2)
- D3 pad 2: Net-(C10-Pad2) -> Net-(B1-Pad1)
- D4 pad 1: Net-(B1-Pad1) -> Net-(C10-Pad2)
- D4 pad 2: Net-(C10-Pad2) -> Net-(B1-Pad1)
- D5 pad 1: Net-(C3-Pad1) -> Net-(C10-Pad2)
- D5 pad 2: Net-(C10-Pad2) -> Net-(C3-Pad1)
- D6 pad 1: Net-(C3-Pad1) -> Net-(C10-Pad2)
- D6 pad 2: Net-(C10-Pad2) -> Net-(C3-Pad1)
- D7 pad 1: Net-(C14-Pad2) -> Net-(C10-Pad2)
- D7 pad 2: Net-(C10-Pad2) -> Net-(C14-Pad2)
- Q12 pad 1: Net-(Q12-Pad1) -> /A1
- Q5 pad 3: /Q3_G -> Net-(D14-Pad2)
- R16 pad 2: Net-(C28-Pad1) -> /A1
- R19 pad 2: Net-(D14-Pad1) -> /Q3_G
- R38 pad 2: Net-(Q12-Pad1) -> /A1
- R40 pad 1: Net-(Q12-Pad1) -> /A1
- R40 pad 2: /A1 -> Net-(Q12-Pad2)
- U1 pad 1: Net-(U1-Pad1) -> Net-(Q7-Pad3)
- U1 pad 12: Net-(U1-Pad12) -> Net-(R23-Pad1)
- U1 pad 14: Net-(C28-Pad1) -> /A1
- U1 pad 2: Net-(U1-Pad12) -> Net-(R23-Pad1)
- U100 pad 3: /A2 -> /G2
- U2 pad 1: Net-(U2-Pad1) -> Net-(C55-Pad1)
- U2 pad 11: Net-(U2-Pad11) -> Net-(R23-Pad1)
- U2 pad 12: Net-(U2-Pad1) -> Net-(C55-Pad1)
- U2 pad 13: Net-(U2-Pad1) -> Net-(C55-Pad1)
- U2 pad 14: Net-(C28-Pad1) -> /A1
- U2 pad 2: Net-(U2-Pad1) -> Net-(C55-Pad1)
- U3 pad 14: Net-(C28-Pad1) -> /A1
- U4 pad 4: Net-(C28-Pad1) -> /A1
- U6 pad 14: Net-(C28-Pad1) -> /A1
Routing:
- net GND: track 0.00 -> 1883.3 mm, vias 0 -> 1
- net /A1: track 0.00 -> 457.2 mm
- net /G2: track 0.00 -> 371.3 mm
- net /A4: track 0.00 -> 346.1 mm
- net /A2: track 0.00 -> 341.4 mm
- net Net-(C10-Pad2): track 0.00 -> 280.9 mm
- net Net-(D25-Pad2): track 0.00 -> 184.8 mm
- net Net-(B1-Pad1): track 0.00 -> 158.2 mm
- net Net-(R4-Pad1): track 0.00 -> 152.4 mm
- net Net-(C3-Pad1): track 0.00 -> 143.3 mm
- net /Q3_G: track 0.00 -> 131.0 mm
- net Net-(A11-Pad1): track 0.00 -> 123.4 mm
- net Net-(C39-Pad2): track 0.00 -> 112.0 mm
- net Net-(C36-Pad1): track 0.00 -> 99.6 mm
- net Net-(R22-Pad2): track 0.00 -> 94.8 mm
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
Commit message: update layout
Connections:
- C44 pad 1: Net-(C44-Pad1) -> GND
- C45 pad 1: Net-(C44-Pad1) -> GND
- C49 pad 1: Net-(C44-Pad1) -> GND
- Q9 pad 1: Net-(C44-Pad1) -> GND
- R31 pad 1: Net-(C44-Pad1) -> GND
- R41 pad 1: Net-(R41-Pad1) -> Net-(C50-Pad2)
- R42 pad 2: Net-(R41-Pad1) -> Net-(C50-Pad2)
Routing:
- net /A1: track 457.2 -> 790.1 mm
- net /-Valim: track 25.9 -> 298.5 mm
- net GND: track 1883.3 -> 2039.5 mm
- net Net-(R64-Pad2): track 0.00 -> 122.0 mm, vias 0 -> 2
- net Net-(A5-Pad1): track 5.00 -> 122.3 mm
- net Net-(C15-Pad2): track 0.00 -> 93.8 mm
- net Net-(D16-Pad2): track 36.0 -> 116.1 mm
- net Net-(Q7-Pad3): track 76.9 -> 145.1 mm
- net Net-(A12-Pad1): track 0.00 -> 59.2 mm
- net Net-(A10-Pad1): track 10.6 -> 64.2 mm
- net Net-(A9-Pad1): track 5.50 -> 53.6 mm
- net Net-(Q11-Pad3): track 11.6 -> 59.4 mm
- net Net-(R69-Pad1): track 13.7 -> 56.9 mm
- net Net-(C50-Pad2): track 41.3 -> 82.9 mm
- net Net-(R6-Pad1): track 0.00 -> 40.7 mm
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
Commit message: Finish layout
Connections:
- C51 pad 2: Net-(C51-Pad2) -> /-Valim
- R42 pad 1: Net-(C51-Pad2) -> /-Valim
- R45 pad 1: Net-(C51-Pad2) -> /-Valim
- R50 pad 1: Net-(C51-Pad2) -> /-Valim
- R59 pad 2: Net-(C51-Pad2) -> /-Valim
- U3 pad 4: Net-(U3-Pad4) -> Net-(R4-Pad1)
- U3 pad 6: Net-(U3-Pad6) -> Net-(C38-Pad2)
- U3 pad 8: Net-(U3-Pad4) -> Net-(R4-Pad1)
- U4 pad 11: Net-(C51-Pad2) -> /-Valim
- U5 pad 11: Net-(C51-Pad2) -> /-Valim
- U6 pad 1: Net-(U3-Pad4) -> Net-(R4-Pad1)
- U6 pad 9: Net-(U3-Pad6) -> Net-(C38-Pad2)
Routing:
- net /A1: track 790.1 -> 915.1 mm
- net /-Valim: track 298.5 -> 422.7 mm
- net Net-(A6-Pad1): track 17.8 -> 135.7 mm
- net GND: track 2039.5 -> 2147.2 mm
- net Net-(R4-Pad1): track 152.4 -> 247.0 mm
- net Net-(C38-Pad2): track 22.8 -> 89.5 mm
- net Net-(C51-Pad2): track 56.3 -> 0.00 mm
- net Net-(R48-Pad2): track 51.8 -> 97.2 mm
- net Net-(D27-Pad1): track 0.00 -> 41.1 mm
- net Net-(C62-Pad1): track 6.60 -> 30.0 mm
- net Net-(C54-Pad2): track 11.4 -> 34.4 mm
- net Net-(U3-Pad6): track 22.1 -> 0.00 mm
- net Net-(C33-Pad2): track 60.7 -> 79.5 mm
- net Net-(C39-Pad2): track 112.0 -> 129.7 mm
- net Net-(R27-Pad1): track 0.00 -> 15.0 mm
Other:
- board text added: "A"
- board text added: "A1"
- board text added: "A10"
- board text added: "A11"
- board text added: "A12"
- board text added: "A13"
- board text added: "A14"
- board text added: "A15"
- board text added: "A2"
- board text added: "A3"
- board text added: "A4"
- board text added: "A5"
- board text added: "A6"
- board text added: "A7"
- board text added: "A8"
- board text added: "A9"
- board text added: "B1"
- board text added: "B2"
- board text added: "C"
- board text added: "D"
- board text added: "E1"
- board text added: "E2"
- board text added: "F"
- board text added: "G1"
- board text added: "G2"
- board text added: "H"
