File: Breakout_STM32WB/Breakout_QFN48/Breakout_QFN48.kicad_pcb (KiCad board)
At the start: 4 copper layers, 24 x 33.8 mm, 114 parts, among them J1 Debug conn, J10 Conn_01x01, J11 Conn_01x01, J12 Conn_01x01, J13 Conn_01x01, J14 Conn_01x01, J15 Conn_01x01, J16 Conn_01x01, J17 Conn_01x01, J18 Conn_01x01, J19 Conn_01x01, J2 Conn_01x01, J20 Conn_01x01, J21 Conn_01x01, J22 Conn_01x01, J23 Conn_01x01, J24 Conn_01x01, J25 Conn_01x01, J26 Conn_01x01, J27 Conn_01x01, J28 Conn_01x01, J29 Conn_01x01, J3 Conn_01x01, J30 Conn_01x01, J31 Conn_01x01, J32 Conn_01x01, J33 Conn_01x01, J34 Conn_01x01, J35 Conn_01x01, J36 Conn_01x01, J37 Conn_01x01, J38 Conn_01x01, J39 Conn_01x01, J4 Conn_01x01, J40 Conn_01x01, J41 Conn_01x01, J42 Conn_01x01, J43 Conn_01x01, J44 Conn_01x01, J45 Conn_01x01, J46 Conn_01x01, J47 Conn_01x01, J48 Conn_01x01, J5 Conn_01x01, J6 Conn_01x01, J7 Conn_01x01, J8 Conn_01x01, J9 Conn_01x01, SW1 Reset, U1 STM32WB55Cx, U2 LFL212G45TC1A007, U3 MCP1700-3302E_SOT23, Y1 NX2012SA_32-768kHz, Y2 NX2016_32M

Commit message: fix boot0 pull resistor
Routing:
- net GND: vias 91 -> 93

Commit message: Update lib : add VN7003ALH
Parts:
- C19: value 4,7u -> 4.7u
Connections:
- R2 pad 1: +3V3 -> GND
Routing:
- net GND: track 58.1 -> 58.7 mm, vias 93 -> 94
- net +3V3: track 36.0 -> 35.4 mm, vias 10 -> 9
Changed lines of the file:
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@@
   (layers
     (0 F.Cu signal)
-    (1 GND.Cu signal)
-    (2 PWR.Cu signal)
+    (1 GND.Cu signal hide)
+    (2 PWR.Cu signal hide)
     (31 B.Cu signal)
     (32 B.Adhes user)
@@
       (effects (font (size 1 1) (thickness 0.15)))
     )
-    (fp_text value 4,7u (at 0 1.16 90) (layer F.Fab)
+    (fp_text value 4.7u (at 0 1.16 90) (layer F.Fab)
       (effects (font (size 1 1) (thickness 0.15)))
     )
@@
     (fp_line (start 0.46 0.23) (end 0.26 0.23) (layer F.SilkS) (width 0.05))
     (pad 1 smd rect (at -0.275 0) (size 0.3 0.4) (layers F.Cu F.Paste F.Mask)
-      (net 4 +3V3))
+      (net 2 GND))
     (pad 2 smd rect (at 0.275 0) (size 0.3 0.4) (layers F.Cu F.Paste F.SilkS F.Mask)
       (net 49 /BOOT0))
@@
   (via (at 118.589 108.218) (size 0.4) (drill 0.2) (layers F.Cu B.Cu) (net 2))
   (via (at 107.413 103.9635) (size 0.4) (drill 0.2) (layers F.Cu B.Cu) (net 2))
+  (segment (start 122.3 108.475) (end 122.175 108.6) (width 0.15) (layer F.Cu) (net 2))
+  (via (at 122.175 108.575) (size 0.4) (drill 0.2) (layers F.Cu B.Cu) (net 2))
+  (segment (start 122.3 108.1) (end 122.3 108.475) (width 0.15) (layer F.Cu) (net 2))
   (segment (start 109.45 101.625) (end 109.8 101.275) (width 0.15) (layer F.Cu) (net 3))
   (segment (start 109.45 102.07) (end 109.45 101.625) (width 0.15) (layer F.Cu) (net 3))
@@
   (segment (start 112.725 88) (end 112.725 88.65) (width 0.15) (layer F.Cu) (net 4))
   (via (at 112.725 88.65) (size 0.4) (drill 0.2) (layers F.Cu B.Cu) (net 4))
-  (segment (start 122.3 108.475) (end 122.175 108.6) (width 0.15) (layer F.Cu) (net 4))
-  (via (at 122.175 108.575) (size 0.4) (drill 0.2) (layers F.Cu B.Cu) (net 4))
-  (segment (start 122.3 108.1) (end 122.3 108.475) (width 0.15) (layer F.Cu) (net 4))
   (segment (start 122.1815 104.309) (end 122.15 104.2775) (width 0.15) (layer F.Cu) (net 5))
   (segment (start 119.6425 102.58) (end 120.2965 102.58) (width 0.15) (layer F.Cu) (net 5))

Commit message: Update Gas sensor
Routing:
- added copper zone on In2.Cu, net +3V3
- added copper zone on In2.Cu, net +5V
- added copper zone on In1.Cu, net GND
- removed copper zone on PWR.Cu, net +3V3
- removed copper zone on PWR.Cu, net +5V
- removed copper zone on GND.Cu, net GND
Other:
- net class Default removed
