File: Gas_sensor/Gas_sensor.kicad_pcb (KiCad board)
At the start: 4 copper layers, 44.6 x 100.2 mm, 143 parts, among them J1 Conn_02x02_Counter_Clockwise, J2 Conn_01x04, J3 Conn_01x10, J4 Conn_01x01, J5 Conn_01x01, Q1 DMC1229UFDB, Q2 DMC1229UFDB, Q3 Q_NMOS_GSD, Q4 Q_NMOS_GSD, Q5 Q_NMOS_GSD, Q6 Q_NMOS_GSD, SW1 SW_Push, SW10 SW_Push, SW11 SW_Push, SW12 SW_Push, SW2 SW_Push, SW3 SW_Push, SW4 SW_Push, SW5 SW_Push, SW6 SW_Push, SW7 SW_Push, SW8 SW_Push, SW9 SW_Push, U1 LPV511, U10 MCP1700-3302E_SOT23, U11 STM32F401CCUx, U12 TMP117, U13 TPS63070, U14 TPS79333-EP, U15 REG102GA, U2 LPV511, U3 MCP47CMB22, U4 MCP6V71, U5 LPV511, U6 MCP6V71, U7 MCP6V71, U8 MCP6V71, U9 ADS1115IDGS, Y1 25MHz

Commit message: gas sensor : update layout, power missing
Parts:
- moved R17 2.07 mm to (49.6, 64.5), turned to -90 degrees
- moved R19 1.85 mm to (49.6, 65.9), turned to 90 degrees
Connections:
- U11 pad 21: /Sound -> /PW_ON
- U11 pad 26: /Mid -> /Sound
- U11 pad 27: /Low -> /Mid
- U11 pad 28: /PW_ON -> /APO
- U11 pad 39: /APO -> /Low
Routing:
- net /SenseBatt_EN: track 2.30 -> 112.5 mm, vias 1 -> 2
- net /SenseBatt: track 0.95 -> 100.0 mm
- net /Vheater: track 1.93 -> 72.8 mm, vias 0 -> 8
- net /PW_ON: track 1.99 -> 66.0 mm, vias 0 -> 4
- net /SCL: track 0.00 -> 61.4 mm, vias 0 -> 10
- net /SDA: track 0.00 -> 59.9 mm, vias 0 -> 12
- net /SWCLK: track 0.00 -> 52.2 mm, vias 0 -> 4
- net /SWDIO: track 2.45 -> 49.8 mm, vias 0 -> 4
- net /Vref_DAC: track 2.91 -> 29.1 mm, vias 0 -> 4
- net /APO: track 32.4 -> 39.5 mm
- net /Mid: track 14.2 -> 21.1 mm
- net /Low: track 27.1 -> 30.0 mm, vias 2 -> 4
- net /Sound: track 32.9 -> 35.0 mm
- net /High: track 27.0 -> 28.0 mm
- net GND: track 61.7 -> 62.3 mm, vias 7 -> 8

Commit message: gas sensor : update layout, add plane
Parts:
- moved C33 5.85 mm to (44.0, 99.0)
- moved R38 5.85 mm to (43.3, 98.0)
- moved R43 5.85 mm to (42.4, 99.0)
- moved C41 2.89 mm to (54.8, 91.1), turned to 0 degrees
- moved C42 0.94 mm to (54.1, 110.0), turned to -90 degrees
Routing:
- net +9V: track 18.7 -> 104.5 mm, vias 3 -> 9
- net +BATT: track 43.4 -> 97.9 mm
- net +3V3: track 31.5 -> 79.2 mm, vias 8 -> 32
- net GND: track 62.3 -> 100.7 mm, vias 8 -> 54
- net /APO: track 39.5 -> 44.9 mm
- net /SenseBatt_EN: track 112.5 -> 111.6 mm, vias 2 -> 4
- net /SenseBatt: vias 0 -> 2
- added copper zone on In2.Cu, net +3V3
- added copper zone on In2.Cu, net +9V

Commit message: Update Gas sensor
Parts:
- added REF**: MountingHole_2.7mm, MountingHole:MountingHole_2.7mm, F.Cu at (42.6, 133.5)
- added REF**: MountingHole_2.7mm, MountingHole:MountingHole_2.7mm, F.Cu at (70.9, 42.0)
- added REF**: MountingHole_2.7mm, MountingHole:MountingHole_2.7mm, F.Cu at (74.6, 84.3)
- added REF**: MountingHole_2.7mm, MountingHole:MountingHole_2.7mm, F.Cu at (74.6, 43.0)
- added REF**: MountingHole_2.7mm, MountingHole:MountingHole_2.7mm, F.Cu at (40.7, 42.1)
- added REF**: MountingHole_2.7mm, MountingHole:MountingHole_2.7mm, F.Cu at (39.0, 133.5)
- added REF**: MountingHole_2.7mm, MountingHole:MountingHole_2.7mm, F.Cu at (73.2, 133.5)
- added REF**: MountingHole_2.7mm, MountingHole:MountingHole_2.7mm, F.Cu at (37.3, 84.4)
- R10: value R -> 5
- R3, R8: value R -> 10k
- R4: value R -> 5k
- R5: value R -> 82k
- R6: value R -> 100k
- moved R50 0.18 mm to (61.6, 126.6)
- moved C41 0.12 mm to (54.8, 91.2)
Routing:
- net /SenseBatt: track 100.0 -> 104.4 mm
- net /SenseBatt_EN: track 111.6 -> 115.9 mm
- net Net-(R21-Pad2): track 3.15 -> 4.17 mm
- net /PW_ON: track 66.0 -> 65.3 mm
- net Net-(L1-Pad1): track 12.3 -> 13.0 mm
- net Net-(L1-Pad2): track 9.92 -> 10.6 mm
- net GND: vias 54 -> 219
- added copper zone on In2.Cu, net GND

Commit message: Add X-pressure design
Parts:
- R21, R23, R27: value 0 -> nc
- R56: value nc -> 0
- R7, R9: value 0 -> 1k
Changed lines of the file:
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@@
       (effects (font (size 0.6 0.6) (thickness 0.1)) (justify mirror))
     )
-    (fp_text value "nc" (at 0.025 -0.6) (layer "B.Fab") hide
+    (fp_text value "0" (at 0.025 -0.6) (layer "B.Fab") hide
       (effects (font (size 0.25 0.25) (thickness 0.0625)) (justify mirror))
     )
@@
       (effects (font (size 0.6 0.6) (thickness 0.1)) (justify mirror))
     )
-    (fp_text value "0" (at 0.06 0.65) (layer "B.Fab") hide
+    (fp_text value "1k" (at 0.06 0.65) (layer "B.Fab") hide
       (effects (font (size 0.25 0.25) (thickness 0.0625)) (justify mirror))
     )
@@
       (effects (font (size 0.6 0.6) (thickness 0.1)) (justify mirror))
     )
-    (fp_text value "0" (at -1.05 0) (layer "B.Fab") hide
+    (fp_text value "nc" (at -1.05 0) (layer "B.Fab") hide
       (effects (font (size 0.25 0.25) (thickness 0.0625)) (justify mirror))
     )
@@
       (effects (font (size 0.25 0.25) (thickness 0.0625)) (justify mirror))
     )
-    (fp_text user "${REFERENCE}" (at 0 0) (layer "B.Fab")
+    (fp_text user "${REFERENCE}" (at -0.05 0.825) (layer "B.Fab")
       (effects (font (size 0.4 0.4) (thickness 0.1)) (justify mirror))
     )
@@
       (effects (font (size 0.6 0.6) (thickness 0.1)) (justify mirror))
     )
-    (fp_text value "0" (at 0.025 0.65) (layer "B.Fab") hide
+    (fp_text value "nc" (at 0.025 0.65) (layer "B.Fab") hide
       (effects (font (size 0.25 0.25) (thickness 0.0625)) (justify mirror))
     )
@@
       (effects (font (size 0.6 0.6) (thickness 0.1)) (justify mirror))
     )
-    (fp_text value "0" (at -0.05 -0.725) (layer "B.Fab") hide
+    (fp_text value "1k" (at -0.05 -0.725) (layer "B.Fab") hide
       (effects (font (size 0.25 0.25) (thickness 0.0625)) (justify mirror))
     )
@@
       (effects (font (size 0.6 0.6) (thickness 0.1)) (justify mirror))
     )
-    (fp_text value "0" (at 0 -0.6) (layer "B.Fab") hide
-      (effects (font (size 0.25 0.25) (thickness 0.0625)) (justify mirror))
-    )
+    (fp_text value "nc" (at 0 -0.6) (layer "B.Fab") hide
+      (effects (font (size 0.25 0.25) (thickness 0.0625)) (justify mirror))
+    )
